File: Themu/Peripherials.sch (KiCad schematic (older format))
At the start: 16 parts, among them J3 Conn_01x08, U5 MPU-6050

Commit message: Routed completed
Connections:
- net +3V3: now also J3.8 (Pin_8); no longer J3.1 (Pin_1)
- net GND: now also J3.1 (Pin_1); no longer J3.8 (Pin_8)
Other:
- moved on the sheet: J3
Changed lines of the file:
@@
 L Connector_Generic:Conn_01x08 J3
 U 1 1 5F7E9F89
-P 7750 1500
-F 0 "J3" H 7830 1492 50  0000 L CNN
-F 1 "Conn_01x08" H 7830 1401 50  0000 L CNN
-F 2 "Connector_PinHeader_2.54mm:PinHeader_1x08_P2.54mm_Horizontal" H 7750 1500 50  0001 C CNN
-F 3 "https://media.digikey.com/PDF/Data%20Sheets/Sullins%20PDFs/x%20RxCxxxSxxN-M71RC_%2011637-B.pdf" H 7750 1500 50  0001 C CNN
-F 4 "PRPC008SGAN-M71RC" H 7950 1000 50  0000 C CNN "*Digikey"
-	1    7750 1500
-	1    0    0    -1
+P 7650 1750
+F 0 "J3" H 7730 1742 50  0000 L CNN
+F 1 "Conn_01x08" H 7730 1651 50  0000 L CNN
+F 2 "Connector_PinHeader_2.54mm:PinHeader_1x08_P2.54mm_Horizontal" H 7650 1750 50  0001 C CNN
+F 3 "https://media.digikey.com/PDF/Data%20Sheets/Sullins%20PDFs/x%20RxCxxxSxxN-M71RC_%2011637-B.pdf" H 7650 1750 50  0001 C CNN
+F 4 "PRPC008SGAN-M71RC" H 7850 1250 50  0000 C CNN "*Digikey"
+	1    7650 1750
+	-1   0    0    1
 $EndComp
 $Comp
@@
 L power:+3V3 #PWR0103
 U 1 1 5F81646F
-P 7450 1150
-F 0 "#PWR0103" H 7450 1000 50  0001 C CNN
-F 1 "+3V3" H 7465 1323 50  0000 C CNN
-F 2 "" H 7450 1150 50  0001 C CNN
-F 3 "" H 7450 1150 50  0001 C CNN
-	1    7450 1150
+P 7950 1300
+F 0 "#PWR0103" H 7950 1150 50  0001 C CNN
+F 1 "+3V3" H 7965 1473 50  0000 C CNN
+F 2 "" H 7950 1300 50  0001 C CNN
+F 3 "" H 7950 1300 50  0001 C CNN
+	1    7950 1300
 	1    0    0    -1
 $EndComp
@@
 L power:GND #PWR0104
 U 1 1 5F90F590
-P 7450 1950
-F 0 "#PWR0104" H 7450 1700 50  0001 C CNN
-F 1 "GND" H 7455 1777 50  0000 C CNN
-F 2 "" H 7450 1950 50  0001 C CNN
-F 3 "" H 7450 1950 50  0001 C CNN
-	1    7450 1950
+P 7950 2100
+F 0 "#PWR0104" H 7950 1850 50  0001 C CNN
+F 1 "GND" H 7955 1927 50  0000 C CNN
+F 2 "" H 7950 2100 50  0001 C CNN
+F 3 "" H 7950 2100 50  0001 C CNN
+	1    7950 2100
 	1    0    0    -1
 $EndComp
-Text Label 7250 1800 0    50   ~ 0
-BUTTON
-Text Label 7250 1600 0    50   ~ 0
-FLEX4
-Text Label 7250 1500 0    50   ~ 0
-FLEX3
-Text Label 7250 1400 0    50   ~ 0
-FLEX2
-Text Label 7250 1300 0    50   ~ 0
-FLEX1
 Wire Wire Line
-	7450 1150 7450 1200
+	7950 2100 7950 2050
 Wire Wire Line
-	7450 1200 7550 1200
+	7950 2050 7850 2050
 Wire Wire Line
-	7250 1300 7550 1300
+	8150 1950 7850 1950
 Wire Wire Line
-	7550 1400 7250 1400
+	7850 1850 8150 1850
 Wire Wire Line
-	7250 1500 7550 1500
+	8150 1750 7850 1750
 Wire Wire Line
-	7550 1600 7250 1600
+	7850 1650 8150 1650
 Wire Wire Line
-	7250 1700 7550 1700
+	8150 1550 7850 1550
 Wire Wire Line
-	7550 1800 7250 1800
+	7850 1450 8150 1450
 Wire Wire Line
-	7450 1950 7450 1900
+	7950 1300 7950 1350
 Wire Wire Line
-	7450 1900 7550 1900
+	7950 1350 7850 1350
 Wire Notes Line
 	4200 900  8400 900
@@
 Wire Notes Line
 	4200 2550 4200 900
-Text Label 7250 1700 0    50   ~ 0
+Text Label 8150 1750 2    50   ~ 0
+FLEX3
+Text Label 8150 1650 2    50   ~ 0
+FLEX4
+Text Label 8150 1850 2    50   ~ 0
+FLEX2
+Text Label 8150 1550 2    50   ~ 0
 FLEX5
+Text Label 8150 1950 2    50   ~ 0
+FLEX1
+Text Label 8150 1450 2    50   ~ 0
+BUTTON
 $EndSCHEMATC
