File: Themu/Power.sch (KiCad schematic (older format))
At the start: 14 parts, among them J2 Conn_01x02, Q3 DMP2045U, U2 AP2112K-3.3, U4 MCP73831-2-OT

Commit message: Routed completed
Parts:
- renumbered D3 to L2
Changed lines of the file:
@@
 $EndComp
 $Comp
-L Device:LED_Small_ALT D3
+L Device:LED_Small_ALT L2
 U 1 1 5F5F5CC9
 P 6700 1250
-F 0 "D3" V 6800 1100 50  0000 C CNN
+F 0 "L2" V 6800 1100 50  0000 C CNN
 F 1 "RED LED" V 6700 900 50  0000 C CNN
 F 2 "LED_SMD:LED_0603_1608Metric_Pad1.05x0.95mm_HandSolder" V 6700 1250 50  0001 C CNN
