File: Main_Board/Peripherials.sch (KiCad schematic (older format))
At the start: 16 parts, among them J3 Conn_01x08, U5 MPU-6050

Commit message: Partial commit
Parts:
- added R22: 1K, Resistor_SMD:R_0603_1608Metric_Pad1.05x0.95mm_HandSolder, symbol Device:R_Small_US
- R15, R16, R17, R18, R19: value 1K -> 47K; *Arrow (none) -> ERJ-U3RD4702V
Connections:
- net +3V3: now also R15.1, R16.1, R17.1, R18.1, R19.1; no longer J3.8 (Pin_8)
- net BTN: now also R22.2; no longer J3.7 (Pin_7)
- net GND: no longer R15.1, R16.1, R17.1, R18.1, R19.1
- new net BUTTON: J3.7 (Pin_7), R22.1
- no-connect marks 3 -> 4
Other:
- note added: "Cambiar:\nR15,16,17,18,19 por 47K\nc9 por 0.1uf"
- moved on the sheet: C11, C12, R15, R16, R17, R18, R19

Commit message: Rev 2.0 commit. INTI revision.
Parts:
- C9: value 1000pF 25V X5R -> 0.1uF 16V X7R; *Digikey 06033C102KAT2A -> 0603YC104K4T2A
Connections:
- net GND: now also J3.8 (Pin_8); no longer J3.1 (Pin_1)
Other:
- note removed: "Cambiar:\nR15,16,17,18,19 por 47K\nc9 por 0.1uf"
- moved on the sheet: C9, J3, R11, R15, R16, R17, R18, R19, R22

Commit message: Resolving issues. (#9)
- Bottom silk legend changed.
- New tracing rules added for power supply lines.
- D3 led changed for QBLP655R-RGB. 3D model missing.
Parts:
- C10, C11: value 0.1uF 25V X7R -> 0.1uF 100V X7R; *Arrow (none) -> GRM188R72A104KA35D
- C12: *Arrow (none) -> GRM187R60J226ME15D
- C13: value 2200pF 50V X7R -> 0.0022uF 200V X7R; *Arrow (none) -> GRM188R72D222KW07D
- C9: value 0.1uF 16V X7R -> 0.1uF 100V X7R; *Arrow (none) -> GRM188R72A104KA35D
- R11: *Arrow (none) -> RN73R1JTTD1002B25
- R12, R13, R14: *Arrow (none) -> RN731JTTD4701B25
- R15, R16, R17, R18, R19: *Arrow ERJ-U3RD4702V -> RN73R1JTTD4702B25
- R22: *Arrow (none) -> RN731JTTD1001B25; *Digikey CR0603-FX-1002ELF -> CR0603-FX-1001ELF
- U5: *Arrow (none) -> MPU-6050 (QUOTE)
Changed lines of the file:
@@
 P 1200 3250
 F 0 "C10" H 1292 3296 50  0000 L CNN
-F 1 "0.1uF 25V X7R" H 1292 3205 50  0000 L CNN
+F 1 "0.1uF 100V X7R" H 1292 3205 50  0000 L CNN
 F 2 "Capacitor_SMD:C_0603_1608Metric_Pad1.05x0.95mm_HandSolder" H 1200 3250 50  0001 C CNN
-F 3 "http://datasheets.avx.com/X7RDielectric.pdf" H 1200 3250 50  0001 C CNN
+F 3 "https://static6.arrow.com/aropdfconversion/11ff84947bdbed6cecdb5e2db8d31166d37b9d20/grm188r72a104ka35.pdf" H 1200 3250 50  0001 C CNN
 F 4 "06033C104KAT4A" H 1200 3250 50  0001 C CNN "*Digikey"
+F 5 "GRM188R72A104KA35D" H 1200 3250 50  0001 C CNN "*Arrow"
 	1    1200 3250
 	1    0    0    -1
@@
 F 3 "https://invensense.tdk.com/wp-content/uploads/2015/02/MPU-6000-Datasheet1.pdf" H 2450 2300 50  0001 C CNN
 F 4 "1428-1007-1-ND" H 2450 2450 50  0001 C CNN "*Digikey"
+F 5 "MPU-6050 (QUOTE)" H 2450 2450 50  0001 C CNN "*Arrow"
 	1    2450 2450
 	1    0    0    -1
@@
 F 1 "4.7K" H 1268 2405 50  0000 L CNN
 F 2 "Resistor_SMD:R_0603_1608Metric_Pad1.05x0.95mm_HandSolder" H 1200 2450 50  0001 C CNN
-F 3 "https://www.bourns.com/docs/product-datasheets/CRxxxxx.pdf" H 1200 2450 50  0001 C CNN
+F 3 "https://static6.arrow.com/aropdfconversion/bc77abbb940933dbec058fcb6d36cc6b880d3e09/rn73.pdf" H 1200 2450 50  0001 C CNN
 F 4 "CR0603-FX-4701ELF" H 1200 2450 50  0001 C CNN "*Digikey"
+F 5 "RN731JTTD4701B25" H 1200 2450 50  0001 C CNN "*Arrow"
 	1    1200 2450
 	1    0    0    -1
@@
 F 1 "4.7K" H 1168 1855 50  0000 L CNN
 F 2 "Resistor_SMD:R_0603_1608Metric_Pad1.05x0.95mm_HandSolder" H 1100 1900 50  0001 C CNN
-F 3 "https://www.bourns.com/docs/product-datasheets/CRxxxxx.pdf" H 1100 1900 50  0001 C CNN
+F 3 "https://static6.arrow.com/aropdfconversion/bc77abbb940933dbec058fcb6d36cc6b880d3e09/rn73.pdf" H 1100 1900 50  0001 C CNN
 F 4 "CR0603-FX-4701ELF" H 1100 1900 50  0001 C CNN "*Digikey"
+F 5 "RN731JTTD4701B25" H 1100 1900 50  0001 C CNN "*Arrow"
 	1    1100 1900
 	1    0    0    -1
@@
 F 1 "4.7K" H 1468 1855 50  0000 L CNN
 F 2 "Resistor_SMD:R_0603_1608Metric_Pad1.05x0.95mm_HandSolder" H 1400 1900 50  0001 C CNN
-F 3 "https://www.bourns.com/docs/product-datasheets/CRxxxxx.pdf" H 1400 1900 50  0001 C CNN
+F 3 "https://static6.arrow.com/aropdfconversion/bc77abbb940933dbec058fcb6d36cc6b880d3e09/rn73.pdf" H 1400 1900 50  0001 C CNN
 F 4 "CR0603-FX-4701ELF" H 1400 1900 50  0001 C CNN "*Digikey"
+F 5 "RN731JTTD4701B25" H 1400 1900 50  0001 C CNN "*Arrow"
 	1    1400 1900
 	1    0    0    -1
@@
 AR Path="/5F450ACB/5F4C4C76" Ref="C11"  Part="1"
 F 0 "C11" H 2950 1550 50  0000 L CNN
-F 1 "0.1uF 25V X7R" H 3150 1550 50  0000 L CNN
+F 1 "0.1uF 100V X7R" H 3150 1550 50  0000 L CNN
 F 2 "Capacitor_SMD:C_0603_1608Metric_Pad1.05x0.95mm_HandSolder" H 2750 1500 50  0001 C CNN
-F 3 "http://datasheets.avx.com/X7RDielectric.pdf" H 2750 1500 50  0001 C CNN
+F 3 "https://static6.arrow.com/aropdfconversion/11ff84947bdbed6cecdb5e2db8d31166d37b9d20/grm188r72a104ka35.pdf" H 2750 1500 50  0001 C CNN
 F 4 "06033C104KAT4A" H 2750 1500 50  0001 C CNN "*Digikey"
+F 5 "GRM188R72A104KA35D" H 2750 1500 50  0001 C CNN "*Arrow"
 	1    2750 1500
 	1    0    0    -1
@@
 F 1 "22uF 6.3V X5R" H 3200 1600 50  0000 L CNN
 F 2 "Capacitor_SMD:C_0603_1608Metric_Pad1.05x0.95mm_HandSolder" H 2900 1600 50  0001 C CNN
-F 3 "http://datasheets.avx.com/cx5r.pdf" H 2900 1600 50  0001 C CNN
+F 3 "https://static6.arrow.com/aropdfconversion/c523d1a354f6499a24517f7d97f0018db57c5966/grm187r60j226me15.pdf" H 2900 1600 50  0001 C CNN
 F 4 "06036D226MAT2A" H 2900 1600 50  0001 C CNN "*Digikey"
+F 5 "GRM187R60J226ME15D" H 2900 1600 50  0001 C CNN "*Arrow"
 	1    2900 1600
 	1    0    0    -1
@@
 P 6050 1900
 F 0 "C9" H 6150 1850 50  0000 L CNN
-F 1 "0.1uF 16V X7R" H 6150 1750 50  0000 L CNN
+F 1 "0.1uF 100V X7R" H 6150 1750 50  0000 L CNN
 F 2 "Capacitor_SMD:C_0603_1608Metric_Pad1.05x0.95mm_HandSolder" H 6050 1900 50  0001 C CNN
-F 3 "http://datasheets.avx.com/X7RDielectric.pdf" H 6050 1900 50  0001 C CNN
+F 3 "https://static6.arrow.com/aropdfconversion/11ff84947bdbed6cecdb5e2db8d31166d37b9d20/grm188r72a104ka35.pdf" H 6050 1900 50  0001 C CNN
 F 4 "0603YC104K4T2A" H 6050 1900 50  0001 C CNN "*Digikey"
+F 5 "GRM188R72A104KA35D" H 6050 1900 50  0001 C CNN "*Arrow"
 	1    6050 1900
 	1    0    0    -1
@@
 F 1 "10K" H 6118 1455 50  0000 L CNN
 F 2 "Resistor_SMD:R_0603_1608Metric_Pad1.05x0.95mm_HandSolder" H 6050 1500 50  0001 C CNN
-F 3 "https://www.bourns.com/docs/product-datasheets/CRxxxxx.pdf" H 6050 1500 50  0001 C CNN
+F 3 "https://static6.arrow.com/aropdfconversion/662263d61145c0a53f06cbe0deb101d367377ab5/rn73r.pdf" H 6050 1500 50  0001 C CNN
 F 4 "CR0603-FX-1002ELF" H 6050 1500 50  0001 C CNN "*Digikey"
+F 5 "RN73R1JTTD1002B25" H 6050 1500 50  0001 C CNN "*Arrow"
 	1    6050 1500
 	1    0    0    -1
@@
 F 1 "47K" H 4950 2500 50  0000 C CNN
 F 2 "Resistor_SMD:R_0603_1608Metric_Pad1.05x0.95mm_HandSolder" H 5100 2450 50  0001 C CNN
-F 3 "https://www.bourns.com/docs/product-datasheets/CRxxxxx.pdf" H 5100 2450 50  0001 C CNN
+F 3 "https://static6.arrow.com/aropdfconversion/662263d61145c0a53f06cbe0deb101d367377ab5/rn73r.pdf" H 5100 2450 50  0001 C CNN
 F 4 "CR0603-FX-1001ELF" H 5100 2450 50  0001 C CNN "*Digikey"
-F 5 "ERJ-U3RD4702V" H 5100 2450 50  0001 C CNN "*Arrow"
+F 5 "RN73R1JTTD4702B25" H 5100 2450 50  0001 C CNN "*Arrow"
 	1    5100 2450
 	1    0    0    -1
@@
 F 1 "47K" H 4850 2200 50  0000 C CNN
 F 2 "Resistor_SMD:R_0603_1608Metric_Pad1.05x0.95mm_HandSolder" H 5000 2150 50  0001 C CNN
-F 3 "https://www.bourns.com/docs/product-datasheets/CRxxxxx.pdf" H 5000 2150 50  0001 C CNN
+F 3 "https://static6.arrow.com/aropdfconversion/662263d61145c0a53f06cbe0deb101d367377ab5/rn73r.pdf" H 5000 2150 50  0001 C CNN
 F 4 "CR0603-FX-1001ELF" H 5000 2150 50  0001 C CNN "*Digikey"
-F 5 "ERJ-U3RD4702V" H 5000 2150 50  0001 C CNN "*Arrow"
+F 5 "RN73R1JTTD4702B25" H 5000 2150 50  0001 C CNN "*Arrow"
 	1    5000 2150
 	1    0    0    -1
@@
 F 1 "47K" H 4750 1900 50  0000 C CNN
 F 2 "Resistor_SMD:R_0603_1608Metric_Pad1.05x0.95mm_HandSolder" H 4900 1850 50  0001 C CNN
-F 3 "https://www.bourns.com/docs/product-datasheets/CRxxxxx.pdf" H 4900 1850 50  0001 C CNN
+F 3 "https://static6.arrow.com/aropdfconversion/662263d61145c0a53f06cbe0deb101d367377ab5/rn73r.pdf" H 4900 1850 50  0001 C CNN
 F 4 "CR0603-FX-1001ELF" H 4900 1850 50  0001 C CNN "*Digikey"
-F 5 "ERJ-U3RD4702V" H 4900 1850 50  0001 C CNN "*Arrow"
+F 5 "RN73R1JTTD4702B25" H 4900 1850 50  0001 C CNN "*Arrow"
 	1    4900 1850
 	1    0    0    -1
@@
 F 1 "47K" H 4650 1600 50  0000 C CNN
 F 2 "Resistor_SMD:R_0603_1608Metric_Pad1.05x0.95mm_HandSolder" H 4800 1550 50  0001 C CNN
-F 3 "https://www.bourns.com/docs/product-datasheets/CRxxxxx.pdf" H 4800 1550 50  0001 C CNN
+F 3 "https://static6.arrow.com/aropdfconversion/662263d61145c0a53f06cbe0deb101d367377ab5/rn73r.pdf" H 4800 1550 50  0001 C CNN
 F 4 "CR0603-FX-1001ELF" H 4800 1550 50  0001 C CNN "*Digikey"
-F 5 "ERJ-U3RD4702V" H 4800 1550 50  0001 C CNN "*Arrow"
+F 5 "RN73R1JTTD4702B25" H 4800 1550 50  0001 C CNN "*Arrow"
 	1    4800 1550
 	1    0    0    -1
@@
 F 1 "47K" H 4550 1300 50  0000 C CNN
 F 2 "Resistor_SMD:R_0603_1608Metric_Pad1.05x0.95mm_HandSolder" H 4700 1250 50  0001 C CNN
-F 3 "https://www.bourns.com/docs/product-datasheets/CRxxxxx.pdf" H 4700 1250 50  0001 C CNN
+F 3 "https://static6.arrow.com/aropdfconversion/662263d61145c0a53f06cbe0deb101d367377ab5/rn73r.pdf" H 4700 1250 50  0001 C CNN
 F 4 "CR0603-FX-1001ELF" H 4700 1250 50  0001 C CNN "*Digikey"
-F 5 "ERJ-U3RD4702V" H 4700 1250 50  0001 C CNN "*Arrow"
+F 5 "RN73R1JTTD4702B25" H 4700 1250 50  0001 C CNN "*Arrow"
 	1    4700 1250
 	1    0    0    -1
@@
 P 3550 3050
 F 0 "C13" H 3300 3100 50  0000 L CNN
-F 1 "2200pF 50V X7R" H 2800 3000 50  0000 L CNN
+F 1 "0.0022uF 200V X7R" H 2800 3000 50  0000 L CNN
 F 2 "Capacitor_SMD:C_0603_1608Metric_Pad1.05x0.95mm_HandSolder" H 3550 3050 50  0001 C CNN
-F 3 "http://datasheets.avx.com/X7RDielectric.pdf" H 3550 3050 50  0001 C CNN
+F 3 "https://static6.arrow.com/aropdfconversion/242178f0aecc5c9cbdfbc9a722c8bf8d331b61f/grm188r72d222kw07.pdf" H 3550 3050 50  0001 C CNN
 F 4 "06035C222KAT2A" H 3550 3050 50  0001 C CNN "*Digikey"
+F 5 "GRM188R72D222KW07D" H 3550 3050 50  0001 C CNN "*Arrow"
 	1    3550 3050
 	1    0    0    -1
@@
 F 1 "1K" V 6350 1800 50  0000 L CNN
 F 2 "Resistor_SMD:R_0603_1608Metric_Pad1.05x0.95mm_HandSolder" H 6250 1700 50  0001 C CNN
-F 3 "https://www.bourns.com/docs/product-datasheets/CRxxxxx.pdf" H 6250 1700 50  0001 C CNN
-F 4 "CR0603-FX-1002ELF" H 6250 1700 50  0001 C CNN "*Digikey"
+F 3 "https://static6.arrow.com/aropdfconversion/bc77abbb940933dbec058fcb6d36cc6b880d3e09/rn73.pdf" H 6250 1700 50  0001 C CNN
+F 4 "CR0603-FX-1001ELF" H 6250 1700 50  0001 C CNN "*Digikey"
+F 5 "RN731JTTD1001B25" H 6250 1700 50  0001 C CNN "*Arrow"
 	1    6250 1700
 	0    1    1    0

Commit message: Changing I2C pins
Parts:
- C10, C11, C12, C13, C9: symbol Device:C_Small -> Themu-Main-rescue:C_Small-Device
- J3: symbol Connector_Generic:Conn_01x08 -> Themu-Main-rescue:Conn_01x08-Connector_Generic
- R11, R12, R13, R14, R15, R16, R17, R18, R19, R22: symbol Device:R_Small_US -> Themu-Main-rescue:R_Small_US-Device
- U5: symbol Sensor_Motion:MPU-6050 -> Themu-Main-rescue:MPU-6050-Sensor_Motion
Changed lines of the file:
@@
 	1200 3100 1200 3150
 $Comp
-L power:GND #PWR09
+L Themu-Main-rescue:GND-power #PWR09
 U 1 1 5F4C01A2
 P 1200 3500
@@
 $EndComp
 $Comp
-L Device:C_Small C10
+L Themu-Main-rescue:C_Small-Device C10
 U 1 1 5F4BED98
 P 1200 3250
@@
 $EndComp
 $Comp
-L Sensor_Motion:MPU-6050 U5
+L Themu-Main-rescue:MPU-6050-Sensor_Motion U5
 U 1 1 5F4A4F5D
 P 2450 2450
@@
 	1200 2350 1750 2350
 $Comp
-L power:GND #PWR08
+L Themu-Main-rescue:GND-power #PWR08
 U 1 1 5F4DD6D1
 P 1200 2750
@@
 $EndComp
 $Comp
-L Device:R_Small_US R13
+L Themu-Main-rescue:R_Small_US-Device R13
 U 1 1 5F4DCD8D
 P 1200 2450
@@
 	1750 2750 1650 2750
 $Comp
-L power:GND #PWR011
+L Themu-Main-rescue:GND-power #PWR011
 U 1 1 5F4DBAAE
 P 1650 2750
@@
 	1750 2150 1400 2150
 $Comp
-L Device:R_Small_US R12
+L Themu-Main-rescue:R_Small_US-Device R12
 U 1 1 5F4D04E6
 P 1100 1900
@@
 $EndComp
 $Comp
-L Device:R_Small_US R14
+L Themu-Main-rescue:R_Small_US-Device R14
 U 1 1 5F4CFB4F
 P 1400 1900
@@
 	2350 1750 2350 1700
 $Comp
-L Device:C_Small C?
+L Themu-Main-rescue:C_Small-Device C?
 U 1 1 5F4C4C76
 P 2750 1500
@@
 $EndComp
 $Comp
-L Device:C_Small C?
+L Themu-Main-rescue:C_Small-Device C?
 U 1 1 5F4C4C70
 P 2900 1600
@@
 $EndComp
 $Comp
-L power:GND #PWR?
+L Themu-Main-rescue:GND-power #PWR?
 U 1 1 5F4C4C6A
 P 3200 1800
@@
 	2550 1350 2550 1700
 $Comp
-L power:GND #PWR015
+L Themu-Main-rescue:GND-power #PWR015
 U 1 1 5F4BCFBC
 P 3550 3500
@@
 	2450 3150 2450 3500
 $Comp
-L power:GND #PWR012
+L Themu-Main-rescue:GND-power #PWR012
 U 1 1 5F4B905D
 P 2450 3500
@@
 SCL
 $Comp
-L power:+3V3 #PWR010
+L Themu-Main-rescue:+3V3-power #PWR010
 U 1 1 5F70FA0C
 P 1400 1550
@@
 $EndComp
 $Comp
-L power:+3V3 #PWR013
+L Themu-Main-rescue:+3V3-power #PWR013
 U 1 1 5F7115D8
 P 2550 1250
@@
 Flex Sensors + Button
 $Comp
-L Device:C_Small C9
+L Themu-Main-rescue:C_Small-Device C9
 U 1 1 5F60116B
 P 6050 1900
@@
 $EndComp
 $Comp
-L power:GND #PWR031
+L Themu-Main-rescue:GND-power #PWR031
 U 1 1 5F602BE7
 P 6050 2100
@@
 	6050 1300 6050 1400
 $Comp
-L power:+3.3V #PWR030
+L Themu-Main-rescue:+3.3V-power #PWR030
 U 1 1 5F602632
 P 6050 1300
@@
 $EndComp
 $Comp
-L Device:R_Small_US R11
+L Themu-Main-rescue:R_Small_US-Device R11
 U 1 1 5F600E2F
 P 6050 1500
@@
 FLX1
 $Comp
-L Device:R_Small_US R15
+L Themu-Main-rescue:R_Small_US-Device R15
 U 1 1 5F7336DD
 P 5100 2450
@@
 FLX2
 $Comp
-L Device:R_Small_US R16
+L Themu-Main-rescue:R_Small_US-Device R16
 U 1 1 5F73D12E
 P 5000 2150
@@
 FLX3
 $Comp
-L Device:R_Small_US R17
+L Themu-Main-rescue:R_Small_US-Device R17
 U 1 1 5F743EE1
 P 4900 1850
@@
 FLX4
 $Comp
-L Device:R_Small_US R18
+L Themu-Main-rescue:R_Small_US-Device R18
 U 1 1 5F7464EA
 P 4800 1550
@@
 FLX5
 $Comp
-L Device:R_Small_US R19
+L Themu-Main-rescue:R_Small_US-Device R19
 U 1 1 5F748D84
 P 4700 1250
@@
 $EndComp
 $Comp
-L Device:C_Small C13
+L Themu-Main-rescue:C_Small-Device C13
 U 1 1 5F4BA235
 P 3550 3050
@@
 BUTTON
 $Comp
-L power:+3.3V #PWR05
+L Themu-Main-rescue:+3.3V-power #PWR05
 U 1 1 5F9E05D4
 P 5150 1150
@@
 	5100 2600 5400 2600
 $Comp
-L Device:R_Small_US R22
+L Themu-Main-rescue:R_Small_US-Device R22
 U 1 1 5FA0B3D0
 P 6250 1700
@@
 	7200 1400 7300 1400
 $Comp
-L power:GND #PWR0104
+L Themu-Main-rescue:GND-power #PWR0104
 U 1 1 5F90F590
 P 7200 2100
@@
 $EndComp
 $Comp
-L Connector_Generic:Conn_01x08 J3
+L Themu-Main-rescue:Conn_01x08-Connector_Generic J3
 U 1 1 5F7E9F89
 P 7500 1700

Commit message: Changing I2C pins (continue)
Parts:
- C10, C11, C12, C13, C9: symbol Themu-Main-rescue:C_Small-Device -> Device:C_Small
- J3: symbol Themu-Main-rescue:Conn_01x08-Connector_Generic -> Connector_Generic:Conn_01x08
- R11, R12, R13, R14, R15, R16, R17, R18, R19, R22: symbol Themu-Main-rescue:R_Small_US-Device -> Device:R_Small_US
- U5: symbol Themu-Main-rescue:MPU-6050-Sensor_Motion -> Sensor_Motion:MPU-6050
Changed lines of the file:
@@
 	1200 3100 1200 3150
 $Comp
-L Themu-Main-rescue:GND-power #PWR09
+L power:GND #PWR09
 U 1 1 5F4C01A2
 P 1200 3500
@@
 $EndComp
 $Comp
-L Themu-Main-rescue:C_Small-Device C10
+L Device:C_Small C10
 U 1 1 5F4BED98
 P 1200 3250
@@
 $EndComp
 $Comp
-L Themu-Main-rescue:MPU-6050-Sensor_Motion U5
+L Sensor_Motion:MPU-6050 U5
 U 1 1 5F4A4F5D
 P 2450 2450
@@
 	1200 2350 1750 2350
 $Comp
-L Themu-Main-rescue:GND-power #PWR08
+L power:GND #PWR08
 U 1 1 5F4DD6D1
 P 1200 2750
@@
 $EndComp
 $Comp
-L Themu-Main-rescue:R_Small_US-Device R13
+L Device:R_Small_US R13
 U 1 1 5F4DCD8D
 P 1200 2450
@@
 	1750 2750 1650 2750
 $Comp
-L Themu-Main-rescue:GND-power #PWR011
+L power:GND #PWR011
 U 1 1 5F4DBAAE
 P 1650 2750
@@
 	1750 2150 1400 2150
 $Comp
-L Themu-Main-rescue:R_Small_US-Device R12
+L Device:R_Small_US R12
 U 1 1 5F4D04E6
 P 1100 1900
@@
 $EndComp
 $Comp
-L Themu-Main-rescue:R_Small_US-Device R14
+L Device:R_Small_US R14
 U 1 1 5F4CFB4F
 P 1400 1900
@@
 	2350 1750 2350 1700
 $Comp
-L Themu-Main-rescue:C_Small-Device C?
+L Device:C_Small C?
 U 1 1 5F4C4C76
 P 2750 1500
@@
 $EndComp
 $Comp
-L Themu-Main-rescue:C_Small-Device C?
+L Device:C_Small C?
 U 1 1 5F4C4C70
 P 2900 1600
@@
 $EndComp
 $Comp
-L Themu-Main-rescue:GND-power #PWR?
+L power:GND #PWR?
 U 1 1 5F4C4C6A
 P 3200 1800
@@
 	2550 1350 2550 1700
 $Comp
-L Themu-Main-rescue:GND-power #PWR015
+L power:GND #PWR015
 U 1 1 5F4BCFBC
 P 3550 3500
@@
 	2450 3150 2450 3500
 $Comp
-L Themu-Main-rescue:GND-power #PWR012
+L power:GND #PWR012
 U 1 1 5F4B905D
 P 2450 3500
@@
 SCL
 $Comp
-L Themu-Main-rescue:+3V3-power #PWR010
+L power:+3V3 #PWR010
 U 1 1 5F70FA0C
 P 1400 1550
@@
 $EndComp
 $Comp
-L Themu-Main-rescue:+3V3-power #PWR013
+L power:+3V3 #PWR013
 U 1 1 5F7115D8
 P 2550 1250
@@
 Flex Sensors + Button
 $Comp
-L Themu-Main-rescue:C_Small-Device C9
+L Device:C_Small C9
 U 1 1 5F60116B
 P 6050 1900
@@
 $EndComp
 $Comp
-L Themu-Main-rescue:GND-power #PWR031
+L power:GND #PWR031
 U 1 1 5F602BE7
 P 6050 2100
@@
 	6050 1300 6050 1400
 $Comp
-L Themu-Main-rescue:+3.3V-power #PWR030
+L power:+3.3V #PWR030
 U 1 1 5F602632
 P 6050 1300
@@
 $EndComp
 $Comp
-L Themu-Main-rescue:R_Small_US-Device R11
+L Device:R_Small_US R11
 U 1 1 5F600E2F
 P 6050 1500
@@
 FLX1
 $Comp
-L Themu-Main-rescue:R_Small_US-Device R15
+L Device:R_Small_US R15
 U 1 1 5F7336DD
 P 5100 2450
@@
 FLX2
 $Comp
-L Themu-Main-rescue:R_Small_US-Device R16
+L Device:R_Small_US R16
 U 1 1 5F73D12E
 P 5000 2150
@@
 FLX3
 $Comp
-L Themu-Main-rescue:R_Small_US-Device R17
+L Device:R_Small_US R17
 U 1 1 5F743EE1
 P 4900 1850
@@
 FLX4
 $Comp
-L Themu-Main-rescue:R_Small_US-Device R18
+L Device:R_Small_US R18
 U 1 1 5F7464EA
 P 4800 1550
@@
 FLX5
 $Comp
-L Themu-Main-rescue:R_Small_US-Device R19
+L Device:R_Small_US R19
 U 1 1 5F748D84
 P 4700 1250
@@
 $EndComp
 $Comp
-L Themu-Main-rescue:C_Small-Device C13
+L Device:C_Small C13
 U 1 1 5F4BA235
 P 3550 3050
@@
 BUTTON
 $Comp
-L Themu-Main-rescue:+3.3V-power #PWR05
+L power:+3.3V #PWR05
 U 1 1 5F9E05D4
 P 5150 1150
@@
 	5100 2600 5400 2600
 $Comp
-L Themu-Main-rescue:R_Small_US-Device R22
+L Device:R_Small_US R22
 U 1 1 5FA0B3D0
 P 6250 1700
@@
 	7200 1400 7300 1400
 $Comp
-L Themu-Main-rescue:GND-power #PWR0104
+L power:GND #PWR0104
 U 1 1 5F90F590
 P 7200 2100
@@
 $EndComp
 $Comp
-L Themu-Main-rescue:Conn_01x08-Connector_Generic J3
+L Connector_Generic:Conn_01x08 J3
 U 1 1 5F7E9F89
 P 7500 1700
