File: Main_Board/ESP32-WROOM-32.sch (KiCad schematic (older format))
At the start: 19 parts, among them J1 USB_B_Micro, Q1 mmbt2222, Q2 mmbt2222, U1 CP2104, U3 ESP32-WROOM-32

Commit message: Changed tracks routing to fit new design rules. Components placement remain the same.
New design rules:
Clearance from 6 mils (0.15 mm) to 8 mils (0.2 mm)
Via Drill/Size from 12/25 mils (0.3/0.635 mm) to 15.74/31.5 mils (0.4/0.8 mm)
Thermal spoke width from 8 mils (0.2 mm) to 11.8 mils (0.3 mm)
Parts:
- L1: footprint Themu_FP_Lib:LED APTF1616LSEEZGKQBKC -> Themu_FP_Lib:LED_APTF1616LSEEZGKQBKC
Changed lines of the file:
@@
 F 0 "L1" H 1300 3383 50  0000 C CNN
 F 1 "LED_ARGB" H 1300 3474 50  0000 C CNN
-F 2 "Themu_FP_Lib:LED APTF1616LSEEZGKQBKC" H 1300 3800 50  0001 C CNN
+F 2 "Themu_FP_Lib:LED_APTF1616LSEEZGKQBKC" H 1300 3800 50  0001 C CNN
 F 3 "https://www.kingbrightusa.com/images/catalog/SPEC/APTF1616LSEEZGKQBKC.pdf" H 1300 3800 50  0001 C CNN
 F 4 "APTF1616LSEEZGKQBKC" H 1300 3850 50  0001 C CNN "*Digikey"

Commit message: Added adapter board for 5 flex sensors and 1 button
Parts:
- L1: footprint Themu_FP_Lib:LED_APTF1616LSEEZGKQBKC -> Main_Board:LED_APTF1616LSEEZGKQBKC
Changed lines of the file:
@@
 F 0 "L1" H 1300 3383 50  0000 C CNN
 F 1 "LED_ARGB" H 1300 3474 50  0000 C CNN
-F 2 "Themu_FP_Lib:LED_APTF1616LSEEZGKQBKC" H 1300 3800 50  0001 C CNN
+F 2 "Main_Board:LED_APTF1616LSEEZGKQBKC" H 1300 3800 50  0001 C CNN
 F 3 "https://www.kingbrightusa.com/images/catalog/SPEC/APTF1616LSEEZGKQBKC.pdf" H 1300 3800 50  0001 C CNN
 F 4 "APTF1616LSEEZGKQBKC" H 1300 3850 50  0001 C CNN "*Digikey"

Commit message: Rev 2.0 commit. INTI revision.
Parts:
- renumbered L1 to D3
Changed lines of the file:
@@
 Date "2020-09-24"
 Rev "02"
-Comp ""
+Comp "By Castro Germán & Diaz Manuel"
 Comment1 ""
 Comment2 ""
@@
 NoConn ~ 3400 2450
 $Comp
-L Device:LED_ARGB L1
+L Device:LED_ARGB D3
 U 1 1 5F8899CA
 P 1300 3850
-F 0 "L1" H 1300 3383 50  0000 C CNN
+F 0 "D3" H 1300 3383 50  0000 C CNN
 F 1 "LED_ARGB" H 1300 3474 50  0000 C CNN
 F 2 "Main_Board:LED_APTF1616LSEEZGKQBKC" H 1300 3800 50  0001 C CNN

Commit message: Resolving issues. (#9)
- Bottom silk legend changed.
- New tracing rules added for power supply lines.
- D3 led changed for QBLP655R-RGB. 3D model missing.
Parts:
- removed D3: LED_ARGB, Main_Board:LED_APTF1616LSEEZGKQBKC, symbol Device:LED_ARGB
- added D3: LED_RABG, Main_Board:LED_QBLP655R_RGB, symbol Device:LED_RABG
- C1, C5, C6: value 0.1uF 25V X7R -> 0.1uF 100V X7R; *Arrow (none) -> GRM188R72A104KA35D
- C14: value 10uF 25V X7R -> 10uF 6.3V X5R; *Arrow (none) -> GRM188R60J106KE47D
- C7: *Arrow (none) -> GRM187R60J226ME15D
- J1: *Arrow (none) -> 1050170001
- Q1, Q2: *Arrow (none) -> MMBT2222LT1G
- R1, R10, R2: *Arrow (none) -> RN73R1JTTD1002B25
- R20: value 1K -> 374R; *Arrow (none) -> RK73H1JTTD3740F
- R21: value 1K -> 232R; *Arrow (none) -> RK73H1JTTD2320F
- R3: value 1K -> 560R; *Arrow (none) -> RK73B1JTTDD561J
- R4, R5: *Arrow (none) -> RN73R1JTTD1003B50
- U1: *Arrow (none) -> CP2104-F03-GM (Quote)
Changed lines of the file:
@@
 F 1 "10K" V 8386 2100 50  0000 C CNN
 F 2 "Resistor_SMD:R_0603_1608Metric_Pad1.05x0.95mm_HandSolder" H 8500 2100 50  0001 C CNN
-F 3 "https://www.bourns.com/docs/product-datasheets/CRxxxxx.pdf" H 8500 2100 50  0001 C CNN
+F 3 "https://static6.arrow.com/aropdfconversion/662263d61145c0a53f06cbe0deb101d367377ab5/rn73r.pdf" H 8500 2100 50  0001 C CNN
 F 4 "CR0603-FX-1002ELF" H 8500 2100 50  0001 C CNN "*Digikey"
+F 5 "RN73R1JTTD1002B25" H 8500 2100 50  0001 C CNN "*Arrow"
 	1    8500 2100
 	0    1    1    0
@@
 F 1 "10K" V 8386 1300 50  0000 C CNN
 F 2 "Resistor_SMD:R_0603_1608Metric_Pad1.05x0.95mm_HandSolder" H 8500 1300 50  0001 C CNN
-F 3 "https://www.bourns.com/docs/product-datasheets/CRxxxxx.pdf" H 8500 1300 50  0001 C CNN
+F 3 "https://static6.arrow.com/aropdfconversion/662263d61145c0a53f06cbe0deb101d367377ab5/rn73r.pdf" H 8500 1300 50  0001 C CNN
 F 4 "CR0603-FX-1002ELF" H 8500 1300 50  0001 C CNN "*Digikey"
+F 5 "RN73R1JTTD1002B25" H 8500 1300 50  0001 C CNN "*Arrow"
 	1    8500 1300
 	0    1    1    0
@@
 F 3 "https://www.onsemi.com/pub/Collateral/MMBT2222LT1-D.PDF" H 8900 2100 50  0001 C CNN
 F 4 "MMBT2222ALT1GOSCT-ND" H 8900 2100 50  0001 C CNN "*Digikey"
+F 5 "MMBT2222LT1G" H 8900 2100 50  0001 C CNN "*Arrow"
 	1    8900 2100
 	1    0    0    1
@@
 F 3 "https://www.onsemi.com/pub/Collateral/MMBT2222LT1-D.PDF" H 8900 1300 50  0001 C CNN
 F 4 "MMBT2222ALT1GOSCT-ND" H 8900 1300 50  0001 C CNN "*Digikey"
+F 5 "MMBT2222LT1G" H 8900 1300 50  0001 C CNN "*Arrow"
 	1    8900 1300
 	1    0    0    -1
@@
 F 1 "10K" H 1168 1255 50  0000 L CNN
 F 2 "Resistor_SMD:R_0603_1608Metric_Pad1.05x0.95mm_HandSolder" H 1100 1300 50  0001 C CNN
-F 3 "https://www.bourns.com/docs/product-datasheets/CRxxxxx.pdf" H 1100 1300 50  0001 C CNN
+F 3 "https://static6.arrow.com/aropdfconversion/662263d61145c0a53f06cbe0deb101d367377ab5/rn73r.pdf" H 1100 1300 50  0001 C CNN
 F 4 "CR0603-FX-1002ELF" H 1100 1300 50  0001 C CNN "*Digikey"
+F 5 "RN73R1JTTD1002B25" H 1100 1300 50  0001 C CNN "*Arrow"
 	1    1100 1300
 	1    0    0    -1
@@
 AR Path="/5F4501E0/5F4A14B8" Ref="C5"  Part="1"
 F 0 "C5" H 1192 1646 50  0000 L CNN
-F 1 "0.1uF 25V X7R" H 1192 1555 50  0000 L CNN
+F 1 "0.1uF 100V X7R" H 1192 1555 50  0000 L CNN
 F 2 "Capacitor_SMD:C_0603_1608Metric_Pad1.05x0.95mm_HandSolder" H 1100 1600 50  0001 C CNN
-F 3 "http://datasheets.avx.com/X7RDielectric.pdf" H 1100 1600 50  0001 C CNN
+F 3 "https://static6.arrow.com/aropdfconversion/11ff84947bdbed6cecdb5e2db8d31166d37b9d20/grm188r72a104ka35.pdf" H 1100 1600 50  0001 C CNN
 F 4 "06033C104KAT4A" H 1100 1600 50  0001 C CNN "*Digikey"
+F 5 "GRM188R72A104KA35D" H 1100 1600 50  0001 C CNN "*Arrow"
 	1    1100 1600
 	1    0    0    -1
@@
 F 1 "22uF 6.3V X5R" H 3542 1205 50  0000 L CNN
 F 2 "Capacitor_SMD:C_0603_1608Metric_Pad1.05x0.95mm_HandSolder" H 3450 1250 50  0001 C CNN
-F 3 "http://datasheets.avx.com/cx5r.pdf" H 3450 1250 50  0001 C CNN
+F 3 "https://static6.arrow.com/aropdfconversion/c523d1a354f6499a24517f7d97f0018db57c5966/grm187r60j226me15.pdf" H 3450 1250 50  0001 C CNN
 F 4 "06036D226MAT2A" H 3450 1250 50  0001 C CNN "*Digikey"
+F 5 "GRM187R60J226ME15D" H 3450 1250 50  0001 C CNN "*Arrow"
 	1    3450 1250
 	1    0    0    -1
@@
 AR Path="/5F4501E0/5F4A14D1" Ref="C6"  Part="1"
 F 0 "C6" H 3092 1296 50  0000 L CNN
-F 1 "0.1uF 25V X7R" H 3092 1205 50  0000 L CNN
+F 1 "0.1uF 100V X7R" H 3092 1205 50  0000 L CNN
 F 2 "Capacitor_SMD:C_0603_1608Metric_Pad1.05x0.95mm_HandSolder" H 3000 1250 50  0001 C CNN
-F 3 "http://datasheets.avx.com/X7RDielectric.pdf" H 3000 1250 50  0001 C CNN
+F 3 "https://static6.arrow.com/aropdfconversion/11ff84947bdbed6cecdb5e2db8d31166d37b9d20/grm188r72a104ka35.pdf" H 3000 1250 50  0001 C CNN
 F 4 "06033C104KAT4A" H 3000 1250 50  0001 C CNN "*Digikey"
+F 5 "GRM188R72A104KA35D" H 3000 1250 50  0001 C CNN "*Arrow"
 	1    3000 1250
 	1    0    0    -1
@@
 F 3 "https://www.silabs.com/documents/public/data-sheets/cp2104.pdf" H 6250 3450 50  0001 C CNN
 F 4 "336-4146-1-ND" H 6800 2200 50  0001 C CNN "*Digikey"
+F 5 "CP2104-F03-GM (Quote)" H 6800 2200 50  0001 C CNN "*Arrow"
 	1    6800 2200
 	1    0    0    -1
@@
 P 5350 1350
 F 0 "C1" H 5442 1396 50  0000 L CNN
-F 1 "0.1uF 25V X7R" H 5442 1305 50  0000 L CNN
+F 1 "0.1uF 100V X7R" H 5442 1305 50  0000 L CNN
 F 2 "Capacitor_SMD:C_0603_1608Metric_Pad1.05x0.95mm_HandSolder" H 5350 1350 50  0001 C CNN
-F 3 "http://datasheets.avx.com/X7RDielectric.pdf" H 5350 1350 50  0001 C CNN
+F 3 "https://static6.arrow.com/aropdfconversion/11ff84947bdbed6cecdb5e2db8d31166d37b9d20/grm188r72a104ka35.pdf" H 5350 1350 50  0001 C CNN
 F 4 "06033C104KAT4A" H 5350 1350 50  0001 C CNN "*Digikey"
+F 5 "GRM188R72A104KA35D" H 5350 1350 50  0001 C CNN "*Arrow"
 	1    5350 1350
 	1    0    0    -1
@@
 F 3 "https://www.molex.com/pdm_docs/sd/1050170001_sd.pdf" H 4900 2750 50  0001 C CNN
 F 4 "1050170001" H 4750 2800 50  0001 C CNN "*Digikey"
+F 5 "1050170001" H 4750 2800 50  0001 C CNN "*Arrow"
 	1    4750 2800
 	1    0    0    -1
@@
 F 1 "100K" H 1168 2305 50  0000 L CNN
 F 2 "Resistor_SMD:R_0603_1608Metric_Pad1.05x0.95mm_HandSolder" H 1100 2350 50  0001 C CNN
-F 3 "https://www.bourns.com/docs/product-datasheets/CRxxxxx.pdf" H 1100 2350 50  0001 C CNN
+F 3 "https://static6.arrow.com/aropdfconversion/662263d61145c0a53f06cbe0deb101d367377ab5/rn73r.pdf" H 1100 2350 50  0001 C CNN
 F 4 "CR0603-FX-1003ELF" H 1100 2350 50  0001 C CNN "*Digikey"
+F 5 "RN73R1JTTD1003B50" H 1100 2350 50  0001 C CNN "*Arrow"
 	1    1100 2350
 	1    0    0    -1
@@
 F 1 "100K" H 1168 2655 50  0000 L CNN
 F 2 "Resistor_SMD:R_0603_1608Metric_Pad1.05x0.95mm_HandSolder" H 1100 2700 50  0001 C CNN
-F 3 "https://www.bourns.com/docs/product-datasheets/CRxxxxx.pdf" H 1100 2700 50  0001 C CNN
+F 3 "https://static6.arrow.com/aropdfconversion/662263d61145c0a53f06cbe0deb101d367377ab5/rn73r.pdf" H 1100 2700 50  0001 C CNN
 F 4 "CR0603-FX-1003ELF" H 1100 2700 50  0001 C CNN "*Digikey"
+F 5 "RN73R1JTTD1003B50" H 1100 2700 50  0001 C CNN "*Arrow"
 	1    1100 2700
 	1    0    0    -1
@@
 P 5150 1600
 F 0 "C14" H 5242 1646 50  0000 L CNN
-F 1 "10uF 25V X7R" H 5242 1555 50  0000 L CNN
+F 1 "10uF 6.3V X5R" H 5242 1555 50  0000 L CNN
 F 2 "Capacitor_SMD:C_1210_3225Metric_Pad1.42x2.65mm_HandSolder" H 5150 1600 50  0001 C CNN
-F 3 "http://datasheets.avx.com/X7RDielectric.pdf" H 5150 1600 50  0001 C CNN
+F 3 "https://static6.arrow.com/aropdfconversion/f7a2596b5312288600ca127f041a86c0cac4c78c/grm188r60j106ke47.pdf" H 5150 1600 50  0001 C CNN
 F 4 "12103C106KAT2A" H 5150 1600 50  0001 C CNN "*Digikey"
+F 5 "GRM188R60J106KE47D" H 5150 1600 50  0001 C CNN "*Arrow"
 	1    5150 1600
 	1    0    0    -1
@@
 P 1650 3650
 F 0 "R3" V 1550 3550 50  0000 C CNN
-F 1 "1K" V 1550 3700 50  0000 C CNN
+F 1 "560R" V 1550 3750 50  0000 C CNN
 F 2 "Resistor_SMD:R_0603_1608Metric_Pad1.05x0.95mm_HandSolder" H 1650 3650 50  0001 C CNN
-F 3 "https://www.bourns.com/docs/product-datasheets/CRxxxxx.pdf" H 1650 3650 50  0001 C CNN
+F 3 "https://static6.arrow.com/aropdfconversion/89b273cd3ad0788d8b71596c5e78488e3c5e22e4/rk73b.pdf" H 1650 3650 50  0001 C CNN
 F 4 "CR0603-FX-1001ELF" H 1650 3650 50  0001 C CNN "*Digikey"
+F 5 "RK73B1JTTDD561J" H 1650 3650 50  0001 C CNN "*Arrow"
 	1    1650 3650
 	0    1    1    0
@@
 P 1650 3850
 F 0 "R20" V 1550 3750 50  0000 C CNN
-F 1 "1K" V 1550 3900 50  0000 C CNN
+F 1 "374R" V 1550 3950 50  0000 C CNN
 F 2 "Resistor_SMD:R_0603_1608Metric_Pad1.05x0.95mm_HandSolder" H 1650 3850 50  0001 C CNN
-F 3 "https://www.bourns.com/docs/product-datasheets/CRxxxxx.pdf" H 1650 3850 50  0001 C CNN
+F 3 "https://static6.arrow.com/aropdfconversion/295cce9d591dbc31ad781a9de7cadb1c39dc0344/rk73h.pdf" H 1650 3850 50  0001 C CNN
 F 4 "CR0603-FX-1001ELF" H 1650 3850 50  0001 C CNN "*Digikey"
+F 5 "RK73H1JTTD3740F" H 1650 3850 50  0001 C CNN "*Arrow"
 	1    1650 3850
 	0    1    1    0
@@
 P 1650 4050
 F 0 "R21" V 1550 3950 50  0000 C CNN
-F 1 "1K" V 1550 4100 50  0000 C CNN
+F 1 "232R" V 1550 4150 50  0000 C CNN
 F 2 "Resistor_SMD:R_0603_1608Metric_Pad1.05x0.95mm_HandSolder" H 1650 4050 50  0001 C CNN
-F 3 "https://www.bourns.com/docs/product-datasheets/CRxxxxx.pdf" H 1650 4050 50  0001 C CNN
+F 3 "https://static6.arrow.com/aropdfconversion/295cce9d591dbc31ad781a9de7cadb1c39dc0344/rk73h.pdf" H 1650 4050 50  0001 C CNN
 F 4 "CR0603-FX-1001ELF" H 1650 4050 50  0001 C CNN "*Digikey"
+F 5 "RK73H1JTTD2320F" H 1650 4050 50  0001 C CNN "*Arrow"
 	1    1650 4050
 	0    1    1    0
@@
 NoConn ~ 3400 2450
 $Comp
-L Device:LED_ARGB D3
-U 1 1 5F8899CA
+L Device:LED_RABG D3
+U 1 1 5FFE32BD
 P 1300 3850
 F 0 "D3" H 1300 3383 50  0000 C CNN
-F 1 "LED_ARGB" H 1300 3474 50  0000 C CNN
-F 2 "Main_Board:LED_APTF1616LSEEZGKQBKC" H 1300 3800 50  0001 C CNN
-F 3 "https://www.kingbrightusa.com/images/catalog/SPEC/APTF1616LSEEZGKQBKC.pdf" H 1300 3800 50  0001 C CNN
-F 4 "APTF1616LSEEZGKQBKC" H 1300 3850 50  0001 C CNN "*Digikey"
+F 1 "LED_RABG" H 1300 3474 50  0000 C CNN
+F 2 "Main_Board:LED_QBLP655R_RGB" H 1300 3800 50  0001 C CNN
+F 3 "https://static6.arrow.com/aropdfconversion/2e9f9b5de02200d8efd894b12d78141ca956a5cd/qblp655-rgb.pdf" H 1300 3800 50  0001 C CNN
+F 4 "QBLP655-RGB" H 1300 3850 50  0001 C CNN "*Arrow"
 	1    1300 3850
 	-1   0    0    1

Commit message: Changing I2C pins
Parts:
- C1, C14, C5, C6, C7: symbol Device:C_Small -> Themu-Main-rescue:C_Small-Device
- D3: symbol Device:LED_RABG -> Themu-Main-rescue:LED_RABG-Device
- J1: symbol Connector:USB_B_Micro -> Themu-Main-rescue:USB_B_Micro-Connector
- Q1, Q2: symbol Device:Q_NPN_EBC -> Themu-Main-rescue:Q_NPN_EBC-Device
- R1, R10, R2, R20, R21, R3, R4, R5: symbol Device:R_Small_US -> Themu-Main-rescue:R_Small_US-Device
- U1: symbol Interface_USB:CP2104 -> Themu-Main-rescue:CP2104-Interface_USB
- U3: symbol RF_Module:ESP32-WROOM-32 -> Themu-Main-rescue:ESP32-WROOM-32-RF_Module
Connections:
- net SCL: now also U3.27 (IO16); no longer U3.22 (SDI/SD1)
- net SDA: now also U3.30 (IO18); no longer U3.21 (SDO/SD0)
Changed lines of the file:
@@
 NoConn ~ 2200 3150
 $Comp
-L power:GND #PWR?
+L Themu-Main-rescue:GND-power #PWR?
 U 1 1 5F4A137A
 P 2800 4350
@@
 NoConn ~ 3400 3150
 NoConn ~ 3400 3050
-NoConn ~ 3400 2950
 NoConn ~ 3400 2850
 NoConn ~ 3400 2650
@@
 	9000 1100 9000 1000
 $Comp
-L Device:R_Small_US R?
+L Themu-Main-rescue:R_Small_US-Device R?
 U 1 1 5F4A13D6
 P 8500 2100
@@
 $EndComp
 $Comp
-L Device:R_Small_US R?
+L Themu-Main-rescue:R_Small_US-Device R?
 U 1 1 5F4A13DC
 P 8500 1300
@@
 $EndComp
 $Comp
-L Device:Q_NPN_EBC Q?
+L Themu-Main-rescue:Q_NPN_EBC-Device Q?
 U 1 1 5F4A13E2
 P 8900 2100
@@
 $EndComp
 $Comp
-L Device:Q_NPN_EBC Q?
+L Themu-Main-rescue:Q_NPN_EBC-Device Q?
 U 1 1 5F4A13E8
 P 8900 1300
@@
 	1100 1400 1100 1500
 $Comp
-L power:GND #PWR?
+L Themu-Main-rescue:GND-power #PWR?
 U 1 1 5F4A14A6
 P 1100 1700
@@
 $EndComp
 $Comp
-L power:+3.3V #PWR?
+L Themu-Main-rescue:+3.3V-power #PWR?
 U 1 1 5F4A14AC
 P 1100 1200
@@
 $EndComp
 $Comp
-L Device:R_Small_US R?
+L Themu-Main-rescue:R_Small_US-Device R?
 U 1 1 5F4A14B2
 P 1100 1300
@@
 $EndComp
 $Comp
-L Device:C_Small C?
+L Themu-Main-rescue:C_Small-Device C?
 U 1 1 5F4A14B8
 P 1100 1600
@@
 	3000 1350 3450 1350
 $Comp
-L power:GND #PWR?
+L Themu-Main-rescue:GND-power #PWR?
 U 1 1 5F4A14C5
 P 3450 1350
@@
 $EndComp
 $Comp
-L Device:C_Small C?
+L Themu-Main-rescue:C_Small-Device C?
 U 1 1 5F4A14CB
 P 3450 1250
@@
 $EndComp
 $Comp
-L Device:C_Small C?
+L Themu-Main-rescue:C_Small-Device C?
 U 1 1 5F4A14D1
 P 3000 1250
@@
 $EndComp
 $Comp
-L power:+3.3V #PWR?
+L Themu-Main-rescue:+3.3V-power #PWR?
 U 1 1 5F4A14D7
 P 2800 1150
@@
 	1    0    0    -1
 $EndComp
-Text HLabel 1950 2950 0    50   BiDi ~ 0
+Text HLabel 3650 2950 2    50   BiDi ~ 0
 SDA
-Text HLabel 1950 3050 0    50   BiDi ~ 0
+Text HLabel 3650 2750 2    50   BiDi ~ 0
 SCL
 Wire Wire Line
-	2200 2950 1950 2950
-Wire Wire Line
-	2200 3050 1950 3050
-$Comp
-L Interface_USB:CP2104 U1
+	3400 2950 3650 2950
+Wire Wire Line
+	3400 2750 3650 2750
+$Comp
+L Themu-Main-rescue:CP2104-Interface_USB U1
 U 1 1 5F606DE2
 P 6800 2200
@@
 $EndComp
 $Comp
-L Device:C_Small C1
+L Themu-Main-rescue:C_Small-Device C1
 U 1 1 5F62B7D9
 P 5350 1350
@@
 $EndComp
 $Comp
-L power:+3.3V #PWR02
+L Themu-Main-rescue:+3.3V-power #PWR02
 U 1 1 5F62C217
 P 5800 1150
@@
 	5800 1150 5800 1250
 $Comp
-L power:GND #PWR?
+L Themu-Main-rescue:GND-power #PWR?
 U 1 1 5F63677B
 P 6800 3450
@@
 Connection ~ 6800 3200
 $Comp
-L Connector:USB_B_Micro J?
+L Themu-Main-rescue:USB_B_Micro-Connector J?
 U 1 1 5F4A152B
 P 4750 2800
@@
 	4650 3200 4750 3200
 $Comp
-L power:GND #PWR?
+L Themu-Main-rescue:GND-power #PWR?
 U 1 1 5F4A149C
 P 4750 3350
@@
 	1100 2450 1100 2550
 $Comp
-L power:GND #PWR?
+L Themu-Main-rescue:GND-power #PWR?
 U 1 1 5F674CFE
 P 1100 2850
@@
 $EndComp
 $Comp
-L Device:R_Small_US R?
+L Themu-Main-rescue:R_Small_US-Device R?
 U 1 1 5F674D0A
 P 1100 2350
@@
 $EndComp
 $Comp
-L Device:R_Small_US R?
+L Themu-Main-rescue:R_Small_US-Device R?
 U 1 1 5F677550
 P 1100 2700
@@
 Connection ~ 1100 2550
 $Comp
-L power:+BATT #PWR06
+L Themu-Main-rescue:+BATT-power #PWR06
 U 1 1 5F67B0FC
 P 1100 2250
@@
 	2200 1750 2100 1750
 $Comp
-L power:VBUS #PWR01
+L Themu-Main-rescue:VBUS-power #PWR01
 U 1 1 5F6AB1E8
 P 5100 2400
@@
 	3400 3750 3850 3750
 $Comp
-L RF_Module:ESP32-WROOM-32 U?
+L Themu-Main-rescue:ESP32-WROOM-32-RF_Module U?
 U 1 1 5F4A1531
 P 2800 2950
@@
 Text HLabel 1750 2050 0    50   Input ~ 0
 FLX1
-NoConn ~ 3400 2750
 Text Label 1550 2550 2    50   ~ 0
 ADC1_CH0
 $Comp
-L Device:C_Small C14
+L Themu-Main-rescue:C_Small-Device C14
 U 1 1 5F7AA131
 P 5150 1600
@@
 $EndComp
 $Comp
-L power:GND #PWR035
+L Themu-Main-rescue:GND-power #PWR035
 U 1 1 5F7AA137
 P 5150 1700
@@
 Connection ~ 5150 1700
 $Comp
-L Device:R_Small_US R3
+L Themu-Main-rescue:R_Small_US-Device R3
 U 1 1 5F857FC9
 P 1650 3650
@@
 $EndComp
 $Comp
-L Device:R_Small_US R20
+L Themu-Main-rescue:R_Small_US-Device R20
 U 1 1 5F858D55
 P 1650 3850
@@
 $EndComp
 $Comp
-L Device:R_Small_US R21
+L Themu-Main-rescue:R_Small_US-Device R21
 U 1 1 5F85AC5C
 P 1650 4050
@@
 $EndComp
 $Comp
-L power:+3.3V #PWR?
+L Themu-Main-rescue:+3.3V-power #PWR?
 U 1 1 5F85EEE7
 P 1100 3350
@@
 NoConn ~ 3400 2450
 $Comp
-L Device:LED_RABG D3
+L Themu-Main-rescue:LED_RABG-Device D3
 U 1 1 5FFE32BD
 P 1300 3850
@@
 	-1   0    0    1
 $EndComp
+NoConn ~ 2200 2950
+NoConn ~ 2200 3050
 $EndSCHEMATC

Commit message: Changing I2C pins (continue)
Parts:
- C1, C14, C5, C6, C7: symbol Themu-Main-rescue:C_Small-Device -> Device:C_Small
- D3: symbol Themu-Main-rescue:LED_RABG-Device -> Device:LED_RABG
- J1: symbol Themu-Main-rescue:USB_B_Micro-Connector -> Connector:USB_B_Micro
- Q1, Q2: symbol Themu-Main-rescue:Q_NPN_EBC-Device -> Device:Q_NPN_EBC
- R1, R10, R2, R20, R21, R3, R4, R5: symbol Themu-Main-rescue:R_Small_US-Device -> Device:R_Small_US
- U1: symbol Themu-Main-rescue:CP2104-Interface_USB -> Interface_USB:CP2104
- U3: symbol Themu-Main-rescue:ESP32-WROOM-32-RF_Module -> RF_Module:ESP32-WROOM-32
Changed lines of the file:
@@
 NoConn ~ 2200 3150
 $Comp
-L Themu-Main-rescue:GND-power #PWR?
+L power:GND #PWR?
 U 1 1 5F4A137A
 P 2800 4350
@@
 	9000 1100 9000 1000
 $Comp
-L Themu-Main-rescue:R_Small_US-Device R?
+L Device:R_Small_US R?
 U 1 1 5F4A13D6
 P 8500 2100
@@
 $EndComp
 $Comp
-L Themu-Main-rescue:R_Small_US-Device R?
+L Device:R_Small_US R?
 U 1 1 5F4A13DC
 P 8500 1300
@@
 $EndComp
 $Comp
-L Themu-Main-rescue:Q_NPN_EBC-Device Q?
+L Device:Q_NPN_EBC Q?
 U 1 1 5F4A13E2
 P 8900 2100
@@
 $EndComp
 $Comp
-L Themu-Main-rescue:Q_NPN_EBC-Device Q?
+L Device:Q_NPN_EBC Q?
 U 1 1 5F4A13E8
 P 8900 1300
@@
 	1100 1400 1100 1500
 $Comp
-L Themu-Main-rescue:GND-power #PWR?
+L power:GND #PWR?
 U 1 1 5F4A14A6
 P 1100 1700
@@
 $EndComp
 $Comp
-L Themu-Main-rescue:+3.3V-power #PWR?
+L power:+3.3V #PWR?
 U 1 1 5F4A14AC
 P 1100 1200
@@
 $EndComp
 $Comp
-L Themu-Main-rescue:R_Small_US-Device R?
+L Device:R_Small_US R?
 U 1 1 5F4A14B2
 P 1100 1300
@@
 $EndComp
 $Comp
-L Themu-Main-rescue:C_Small-Device C?
+L Device:C_Small C?
 U 1 1 5F4A14B8
 P 1100 1600
@@
 	3000 1350 3450 1350
 $Comp
-L Themu-Main-rescue:GND-power #PWR?
+L power:GND #PWR?
 U 1 1 5F4A14C5
 P 3450 1350
@@
 $EndComp
 $Comp
-L Themu-Main-rescue:C_Small-Device C?
+L Device:C_Small C?
 U 1 1 5F4A14CB
 P 3450 1250
@@
 $EndComp
 $Comp
-L Themu-Main-rescue:C_Small-Device C?
+L Device:C_Small C?
 U 1 1 5F4A14D1
 P 3000 1250
@@
 $EndComp
 $Comp
-L Themu-Main-rescue:+3.3V-power #PWR?
+L power:+3.3V #PWR?
 U 1 1 5F4A14D7
 P 2800 1150
@@
 	3400 2750 3650 2750
 $Comp
-L Themu-Main-rescue:CP2104-Interface_USB U1
+L Interface_USB:CP2104 U1
 U 1 1 5F606DE2
 P 6800 2200
@@
 $EndComp
 $Comp
-L Themu-Main-rescue:C_Small-Device C1
+L Device:C_Small C1
 U 1 1 5F62B7D9
 P 5350 1350
@@
 $EndComp
 $Comp
-L Themu-Main-rescue:+3.3V-power #PWR02
+L power:+3.3V #PWR02
 U 1 1 5F62C217
 P 5800 1150
@@
 	5800 1150 5800 1250
 $Comp
-L Themu-Main-rescue:GND-power #PWR?
+L power:GND #PWR?
 U 1 1 5F63677B
 P 6800 3450
@@
 Connection ~ 6800 3200
 $Comp
-L Themu-Main-rescue:USB_B_Micro-Connector J?
+L Connector:USB_B_Micro J?
 U 1 1 5F4A152B
 P 4750 2800
@@
 	4650 3200 4750 3200
 $Comp
-L Themu-Main-rescue:GND-power #PWR?
+L power:GND #PWR?
 U 1 1 5F4A149C
 P 4750 3350
@@
 	1100 2450 1100 2550
 $Comp
-L Themu-Main-rescue:GND-power #PWR?
+L power:GND #PWR?
 U 1 1 5F674CFE
 P 1100 2850
@@
 $EndComp
 $Comp
-L Themu-Main-rescue:R_Small_US-Device R?
+L Device:R_Small_US R?
 U 1 1 5F674D0A
 P 1100 2350
@@
 $EndComp
 $Comp
-L Themu-Main-rescue:R_Small_US-Device R?
+L Device:R_Small_US R?
 U 1 1 5F677550
 P 1100 2700
@@
 Connection ~ 1100 2550
 $Comp
-L Themu-Main-rescue:+BATT-power #PWR06
+L power:+BATT #PWR06
 U 1 1 5F67B0FC
 P 1100 2250
@@
 	2200 1750 2100 1750
 $Comp
-L Themu-Main-rescue:VBUS-power #PWR01
+L power:VBUS #PWR01
 U 1 1 5F6AB1E8
 P 5100 2400
@@
 	3400 3750 3850 3750
 $Comp
-L Themu-Main-rescue:ESP32-WROOM-32-RF_Module U?
+L RF_Module:ESP32-WROOM-32 U?
 U 1 1 5F4A1531
 P 2800 2950
@@
 ADC1_CH0
 $Comp
-L Themu-Main-rescue:C_Small-Device C14
+L Device:C_Small C14
 U 1 1 5F7AA131
 P 5150 1600
@@
 $EndComp
 $Comp
-L Themu-Main-rescue:GND-power #PWR035
+L power:GND #PWR035
 U 1 1 5F7AA137
 P 5150 1700
@@
 Connection ~ 5150 1700
 $Comp
-L Themu-Main-rescue:R_Small_US-Device R3
+L Device:R_Small_US R3
 U 1 1 5F857FC9
 P 1650 3650
@@
 $EndComp
 $Comp
-L Themu-Main-rescue:R_Small_US-Device R20
+L Device:R_Small_US R20
 U 1 1 5F858D55
 P 1650 3850
@@
 $EndComp
 $Comp
-L Themu-Main-rescue:R_Small_US-Device R21
+L Device:R_Small_US R21
 U 1 1 5F85AC5C
 P 1650 4050
@@
 $EndComp
 $Comp
-L Themu-Main-rescue:+3.3V-power #PWR?
+L power:+3.3V #PWR?
 U 1 1 5F85EEE7
 P 1100 3350
@@
 NoConn ~ 3400 2450
 $Comp
-L Themu-Main-rescue:LED_RABG-Device D3
+L Device:LED_RABG D3
 U 1 1 5FFE32BD
 P 1300 3850
