File: Main_Board/Power.sch (KiCad schematic (older format))
At the start: 14 parts, among them J2 Conn_01x02, Q3 DMP2045U, U2 AP2112K-3.3, U4 MCP73831-2-OT

Commit message: Rev 2.0 commit. INTI revision.
Parts:
- renumbered L2 to D1
Other:
- note added: "RPROG\n\n"
- moved on the sheet: C3, C4, C8, D1, R9
Changed lines of the file:
@@
 Date "2020-09-24"
 Rev "02"
-Comp ""
+Comp "By Castro Germán & Diaz Manuel"
 Comment1 ""
 Comment2 ""
@@
 L Device:C_Small C3
 U 1 1 5F5E75DD
-P 3100 2250
-F 0 "C3" H 3192 2296 50  0000 L CNN
-F 1 "10uF 25V X7R" H 3192 2205 50  0000 L CNN
-F 2 "Capacitor_SMD:C_1210_3225Metric_Pad1.42x2.65mm_HandSolder" H 3100 2250 50  0001 C CNN
-F 3 "http://datasheets.avx.com/X7RDielectric.pdf" H 3100 2250 50  0001 C CNN
-F 4 "12103C106KAT2A" H 3100 2250 50  0001 C CNN "*Digikey"
-	1    3100 2250
+P 3100 2350
+F 0 "C3" H 3400 2350 50  0000 L CNN
+F 1 "10uF 25V X7R" H 3550 2350 50  0000 L CNN
+F 2 "Capacitor_SMD:C_1210_3225Metric_Pad1.42x2.65mm_HandSolder" H 3100 2350 50  0001 C CNN
+F 3 "http://datasheets.avx.com/X7RDielectric.pdf" H 3100 2350 50  0001 C CNN
+F 4 "12103C106KAT2A" H 3100 2350 50  0001 C CNN "*Digikey"
+	1    3100 2350
 	1    0    0    -1
 $EndComp
@@
 L Device:C_Small C4
 U 1 1 5F5E8856
-P 3650 2250
-F 0 "C4" H 3742 2296 50  0000 L CNN
-F 1 "1uF 25V X5R" H 3742 2205 50  0000 L CNN
-F 2 "Capacitor_SMD:C_0603_1608Metric_Pad1.05x0.95mm_HandSolder" H 3650 2250 50  0001 C CNN
-F 3 "http://datasheets.avx.com/cx5r.pdf" H 3650 2250 50  0001 C CNN
-F 4 "06033D105KAT2A" H 3650 2250 50  0001 C CNN "*Digikey"
-	1    3650 2250
+P 3300 2200
+F 0 "C4" H 3400 2200 50  0000 L CNN
+F 1 "1uF 25V X5R" H 3550 2200 50  0000 L CNN
+F 2 "Capacitor_SMD:C_0603_1608Metric_Pad1.05x0.95mm_HandSolder" H 3300 2200 50  0001 C CNN
+F 3 "http://datasheets.avx.com/cx5r.pdf" H 3300 2200 50  0001 C CNN
+F 4 "06033D105KAT2A" H 3300 2200 50  0001 C CNN "*Digikey"
+	1    3300 2200
 	1    0    0    -1
 $EndComp
@@
 L power:GND #PWR023
 U 1 1 5F5E8FAE
-P 3650 2500
-F 0 "#PWR023" H 3650 2250 50  0001 C CNN
-F 1 "GND" H 3655 2327 50  0000 C CNN
-F 2 "" H 3650 2500 50  0001 C CNN
-F 3 "" H 3650 2500 50  0001 C CNN
-	1    3650 2500
+P 3300 2500
+F 0 "#PWR023" H 3300 2250 50  0001 C CNN
+F 1 "GND" H 3305 2327 50  0000 C CNN
+F 2 "" H 3300 2500 50  0001 C CNN
+F 3 "" H 3300 2500 50  0001 C CNN
+	1    3300 2500
 	1    0    0    -1
 $EndComp
@@
 L power:+3V3 #PWR022
 U 1 1 5F5E9117
-P 3650 1200
-F 0 "#PWR022" H 3650 1050 50  0001 C CNN
-F 1 "+3V3" H 3665 1373 50  0000 C CNN
-F 2 "" H 3650 1200 50  0001 C CNN
-F 3 "" H 3650 1200 50  0001 C CNN
-	1    3650 1200
+P 3300 1150
+F 0 "#PWR022" H 3300 1000 50  0001 C CNN
+F 1 "+3V3" H 3315 1323 50  0000 C CNN
+F 2 "" H 3300 1150 50  0001 C CNN
+F 3 "" H 3300 1150 50  0001 C CNN
+	1    3300 1150
 	1    0    0    -1
 $EndComp
 Wire Wire Line
 	2900 2000 3100 2000
-Wire Wire Line
-	3650 2000 3650 2150
-Wire Wire Line
-	3100 2000 3100 2150
-Wire Wire Line
-	3100 2350 3100 2500
-Connection ~ 3100 2000
-Wire Wire Line
-	3100 2000 3650 2000
-Wire Wire Line
-	3650 2350 3650 2500
-Wire Wire Line
-	3650 2000 3650 1200
-Connection ~ 3650 2000
 Wire Wire Line
 	2600 2400 2600 2500
@@
 L Device:R_Small_US R9
 U 1 1 5F5F379D
-P 6700 1550
-F 0 "R9" H 6800 1600 50  0000 C CNN
-F 1 "1K" H 6800 1500 50  0000 C CNN
-F 2 "Resistor_SMD:R_0603_1608Metric_Pad1.05x0.95mm_HandSolder" H 6700 1550 50  0001 C CNN
-F 3 "https://www.bourns.com/docs/product-datasheets/CRxxxxx.pdf" H 6700 1550 50  0001 C CNN
-F 4 "CR0603-FX-1001ELF" H 6700 1550 50  0001 C CNN "*Digikey"
-	1    6700 1550
-	1    0    0    -1
-$EndComp
-$Comp
-L Device:LED_Small_ALT L2
+P 6700 1750
+F 0 "R9" H 6800 1800 50  0000 C CNN
+F 1 "1K" H 6800 1700 50  0000 C CNN
+F 2 "Resistor_SMD:R_0603_1608Metric_Pad1.05x0.95mm_HandSolder" H 6700 1750 50  0001 C CNN
+F 3 "https://www.bourns.com/docs/product-datasheets/CRxxxxx.pdf" H 6700 1750 50  0001 C CNN
+F 4 "CR0603-FX-1001ELF" H 6700 1750 50  0001 C CNN "*Digikey"
+	1    6700 1750
+	1    0    0    -1
+$EndComp
+$Comp
+L Device:LED_Small_ALT D1
 U 1 1 5F5F5CC9
-P 6700 1250
-F 0 "L2" V 6800 1100 50  0000 C CNN
-F 1 "RED LED" V 6700 900 50  0000 C CNN
-F 2 "LED_SMD:LED_0603_1608Metric_Pad1.05x0.95mm_HandSolder" V 6700 1250 50  0001 C CNN
-F 3 "https://www.aopled.com/AOP_PDFs/L196L-UEC.pdf" V 6700 1250 50  0001 C CNN
-F 4 "L196L-UEC" H 6700 1250 50  0001 C CNN "*Digikey"
-	1    6700 1250
+P 6700 1500
+F 0 "D1" V 6800 1350 50  0000 C CNN
+F 1 "RED LED" V 6700 1250 50  0000 C CNN
+F 2 "LED_SMD:LED_0603_1608Metric_Pad1.05x0.95mm_HandSolder" V 6700 1500 50  0001 C CNN
+F 3 "https://www.aopled.com/AOP_PDFs/L196L-UEC.pdf" V 6700 1500 50  0001 C CNN
+F 4 "L196L-UEC" H 6700 1500 50  0001 C CNN "*Digikey"
+	1    6700 1500
 	0    -1   -1   0
 $EndComp
@@
 L power:VBUS #PWR027
 U 1 1 5F5FC6D9
-P 6700 1100
-F 0 "#PWR027" H 6700 950 50  0001 C CNN
-F 1 "VBUS" H 6715 1273 50  0000 C CNN
-F 2 "" H 6700 1100 50  0001 C CNN
-F 3 "" H 6700 1100 50  0001 C CNN
-	1    6700 1100
+P 6700 1300
+F 0 "#PWR027" H 6700 1150 50  0001 C CNN
+F 1 "VBUS" H 6715 1473 50  0000 C CNN
+F 2 "" H 6700 1300 50  0001 C CNN
+F 3 "" H 6700 1300 50  0001 C CNN
+	1    6700 1300
 	1    0    0    -1
 $EndComp
@@
 L Device:C_Small C8
 U 1 1 5F5FFAAE
-P 6900 2250
-F 0 "C8" H 6992 2296 50  0000 L CNN
-F 1 "10uF 25V X7R" H 6992 2205 50  0000 L CNN
-F 2 "Capacitor_SMD:C_1210_3225Metric_Pad1.42x2.65mm_HandSolder" H 6900 2250 50  0001 C CNN
-F 3 "http://datasheets.avx.com/X7RDielectric.pdf" H 6900 2250 50  0001 C CNN
-F 4 "12103C106KAT2A" H 6900 2250 50  0001 C CNN "*Digikey"
-	1    6900 2250
+P 6900 2300
+F 0 "C8" H 6992 2346 50  0000 L CNN
+F 1 "10uF 25V X7R" H 6992 2255 50  0000 L CNN
+F 2 "Capacitor_SMD:C_1210_3225Metric_Pad1.42x2.65mm_HandSolder" H 6900 2300 50  0001 C CNN
+F 3 "http://datasheets.avx.com/X7RDielectric.pdf" H 6900 2300 50  0001 C CNN
+F 4 "12103C106KAT2A" H 6900 2300 50  0001 C CNN "*Digikey"
+	1    6900 2300
 	1    0    0    -1
 $EndComp
@@
 L power:GND #PWR029
 U 1 1 5F6012DA
-P 6900 2350
-F 0 "#PWR029" H 6900 2100 50  0001 C CNN
-F 1 "GND" H 6905 2177 50  0000 C CNN
-F 2 "" H 6900 2350 50  0001 C CNN
-F 3 "" H 6900 2350 50  0001 C CNN
-	1    6900 2350
+P 6900 2400
+F 0 "#PWR029" H 6900 2150 50  0001 C CNN
+F 1 "GND" H 6905 2227 50  0000 C CNN
+F 2 "" H 6900 2400 50  0001 C CNN
+F 3 "" H 6900 2400 50  0001 C CNN
+	1    6900 2400
 	1    0    0    -1
 $EndComp
@@
 Text Notes 7250 1700 0    50   ~ 0
 5K = 200mA\n2K = 500mA\n1K = 1000mA\n
-Wire Wire Line
-	6700 2050 6700 1650
-Wire Wire Line
-	6700 1450 6700 1350
-Wire Wire Line
-	6700 1150 6700 1100
-Wire Wire Line
-	6100 1150 6700 1150
-Wire Wire Line
-	6100 1150 6100 1650
-Connection ~ 6700 1150
 $Comp
 L power:+BATT #PWR028
 U 1 1 5F6A9BEF
-P 6900 2050
-F 0 "#PWR028" H 6900 1900 50  0001 C CNN
-F 1 "+BATT" H 6915 2223 50  0000 C CNN
-F 2 "" H 6900 2050 50  0001 C CNN
-F 3 "" H 6900 2050 50  0001 C CNN
-	1    6900 2050
+P 6900 2100
+F 0 "#PWR028" H 6900 1950 50  0001 C CNN
+F 1 "+BATT" H 6915 2273 50  0000 C CNN
+F 2 "" H 6900 2100 50  0001 C CNN
+F 3 "" H 6900 2100 50  0001 C CNN
+	1    6900 2100
 	1    0    0    -1
 $EndComp
@@
 	6500 1850 6600 1850
 Wire Wire Line
-	6600 1850 6600 2150
-Wire Wire Line
-	6600 2150 6900 2150
-Wire Wire Line
-	6900 2050 6900 2150
-Connection ~ 6900 2150
+	6600 2200 6900 2200
+Wire Wire Line
+	6900 2100 6900 2200
+Connection ~ 6900 2200
 $Comp
 L power:PWR_FLAG #FLG0101
@@
 Wire Notes Line
 	750  2900 5200 2900
+Wire Wire Line
+	6100 1650 6550 1650
+Wire Wire Line
+	6600 1850 6600 2200
+Text Notes 7350 1450 0    50   ~ 0
+RPROG\n\n
+Wire Wire Line
+	6700 2050 6700 1850
+Wire Wire Line
+	6700 1650 6700 1600
+Wire Wire Line
+	6700 1400 6700 1350
+Wire Wire Line
+	6550 1650 6550 1350
+Wire Wire Line
+	6550 1350 6700 1350
+Connection ~ 6700 1350
+Wire Wire Line
+	6700 1300 6700 1350
+Wire Wire Line
+	3100 2000 3300 2000
+Wire Wire Line
+	3300 2000 3300 2100
+Wire Wire Line
+	3300 2300 3300 2500
+Connection ~ 3100 2000
+Wire Wire Line
+	3100 2000 3100 2250
+Wire Wire Line
+	3100 2450 3100 2500
+Wire Wire Line
+	3300 1150 3300 2000
+Connection ~ 3300 2000
 $EndSCHEMATC

Commit message: Resolving issues. (#9)
- Bottom silk legend changed.
- New tracing rules added for power supply lines.
- D3 led changed for QBLP655R-RGB. 3D model missing.
Parts:
- C2, C3, C8: value 10uF 25V X7R -> 10uF 6.3V X5R; *Arrow (none) -> GRM188R60J106KE47D
- C4: value 1uF 25V X5R -> 1uF 6.3V X5R; *Arrow (none) -> GRM185R60J105KE26D
- D1: *Arrow (none) -> L196L-UEC-TR
- D2: *Arrow (none) -> MBR120VLSFT3G
- J2: *Arrow (none) -> S2B-PH-K-S(LF)(SN)
- Q3: value DMP2045U -> DMG2305U; *Arrow (none) -> DMG2305UX-13
- R6, R7: *Arrow (none) -> RN73R1JTTD1003B50
- R8: *Arrow (none) -> RN731JTTD4701B25
- R9: *Arrow (none) -> RN731JTTD1001B25
- U2: *Arrow (none) -> AP2112K-3.3TRG1
- U4: *Arrow (none) -> MCP73831T-5ACI/OT
Connections:
- net RegIn: now reaches C2.1, D2.1 (K), Q3.2 (S), R7.1, U2.1 (VIN)
Changed lines of the file:
@@
 F 3 "https://www.diodes.com/assets/Datasheets/AP2112.pdf" H 2600 2200 50  0001 C CNN
 F 4 "AP2112K-3.3TRG1DICT-ND" H 2600 2100 50  0001 C CNN "*Digikey"
+F 5 "AP2112K-3.3TRG1" H 2600 2100 50  0001 C CNN "*Arrow"
 	1    2600 2100
 	1    0    0    -1
@@
 F 1 "100K" V 1800 2100 50  0000 C CNN
 F 2 "Resistor_SMD:R_0603_1608Metric_Pad1.05x0.95mm_HandSolder" H 2000 2100 50  0001 C CNN
-F 3 "https://www.bourns.com/docs/product-datasheets/CRxxxxx.pdf" H 2000 2100 50  0001 C CNN
+F 3 "https://static6.arrow.com/aropdfconversion/662263d61145c0a53f06cbe0deb101d367377ab5/rn73r.pdf" H 2000 2100 50  0001 C CNN
 F 4 "CR0603-FX-1003ELF" H 2000 2100 50  0001 C CNN "*Digikey"
+F 5 "RN73R1JTTD1003B50" H 2000 2100 50  0001 C CNN "*Arrow"
 	1    2000 2100
 	0    -1   -1   0
@@
 F 1 "100K" H 1018 2055 50  0000 L CNN
 F 2 "Resistor_SMD:R_0603_1608Metric_Pad1.05x0.95mm_HandSolder" H 950 2100 50  0001 C CNN
-F 3 "https://www.bourns.com/docs/product-datasheets/CRxxxxx.pdf" H 950 2100 50  0001 C CNN
+F 3 "https://static6.arrow.com/aropdfconversion/662263d61145c0a53f06cbe0deb101d367377ab5/rn73r.pdf" H 950 2100 50  0001 C CNN
 F 4 "CR0603-FX-1003ELF" H 950 2100 50  0001 C CNN "*Digikey"
+F 5 "RN73R1JTTD1003B50" H 950 2100 50  0001 C CNN "*Arrow"
 	1    950  2100
 	1    0    0    -1
@@
 F 1 "MBR120" H 1250 1874 50  0000 C CNN
 F 2 "Diode_SMD:D_SOD-123F" H 1250 1825 50  0001 C CNN
-F 3 "https://www.onsemi.com/pub/Collateral/MBR120VLSFT1-D.PDF" H 1250 2000 50  0001 C CNN
+F 3 "https://static6.arrow.com/aropdfconversion/e8003dfacd77d1ebac96075b6dca1073b845ce4e/mbr120vlsft1-d.pdf" H 1250 2000 50  0001 C CNN
 F 4 "MBR120VLSFT3GOSTR-ND" H 1250 2000 50  0001 C CNN "*Digikey"
+F 5 "MBR120VLSFT3G" H 1250 2000 50  0001 C CNN "*Arrow"
 	1    1250 2000
 	-1   0    0    1
@@
 P 1600 1500
 F 0 "Q3" H 1804 1546 50  0000 L CNN
-F 1 "DMP2045U" H 1804 1455 50  0000 L CNN
+F 1 "DMG2305U" H 1804 1455 50  0000 L CNN
 F 2 "Package_TO_SOT_SMD:SOT-23" H 1800 1425 50  0001 L CIN
-F 3 "https://www.diodes.com/assets/Datasheets/DMP2045U.pdf" H 1600 1500 50  0001 L CNN
+F 3 "https://static6.arrow.com/aropdfconversion/44c9eaa54d5f47022f33e83632b1728195293187/dmg2305ux.pdf" H 1600 1500 50  0001 L CNN
 F 4 "DMP2045U-7DICT-ND" H 1600 1500 50  0001 C CNN "*Digikey"
+F 5 "DMG2305UX-13" H 1600 1500 50  0001 C CNN "*Arrow"
 	1    1600 1500
 	1    0    0    -1
@@
 P 1650 2350
 F 0 "C2" H 1742 2396 50  0000 L CNN
-F 1 "10uF 25V X7R" H 1742 2305 50  0000 L CNN
+F 1 "10uF 6.3V X5R" H 1742 2305 50  0000 L CNN
 F 2 "Capacitor_SMD:C_1210_3225Metric_Pad1.42x2.65mm_HandSolder" H 1650 2350 50  0001 C CNN
-F 3 "http://datasheets.avx.com/X7RDielectric.pdf" H 1650 2350 50  0001 C CNN
+F 3 "https://static6.arrow.com/aropdfconversion/f7a2596b5312288600ca127f041a86c0cac4c78c/grm188r60j106ke47.pdf" H 1650 2350 50  0001 C CNN
 F 4 "12103C106KAT2A" H 1650 2350 50  0001 C CNN "*Digikey"
+F 5 "GRM188R60J106KE47D" H 1650 2350 50  0001 C CNN "*Arrow"
 	1    1650 2350
 	1    0    0    -1
@@
 P 3100 2350
 F 0 "C3" H 3400 2350 50  0000 L CNN
-F 1 "10uF 25V X7R" H 3550 2350 50  0000 L CNN
+F 1 "10uF 6.3V X5R" H 3550 2350 50  0000 L CNN
 F 2 "Capacitor_SMD:C_1210_3225Metric_Pad1.42x2.65mm_HandSolder" H 3100 2350 50  0001 C CNN
-F 3 "http://datasheets.avx.com/X7RDielectric.pdf" H 3100 2350 50  0001 C CNN
+F 3 "https://static6.arrow.com/aropdfconversion/f7a2596b5312288600ca127f041a86c0cac4c78c/grm188r60j106ke47.pdf" H 3100 2350 50  0001 C CNN
 F 4 "12103C106KAT2A" H 3100 2350 50  0001 C CNN "*Digikey"
+F 5 "GRM188R60J106KE47D" H 3100 2350 50  0001 C CNN "*Arrow"
 	1    3100 2350
 	1    0    0    -1
@@
 P 3300 2200
 F 0 "C4" H 3400 2200 50  0000 L CNN
-F 1 "1uF 25V X5R" H 3550 2200 50  0000 L CNN
+F 1 "1uF 6.3V X5R" H 3550 2200 50  0000 L CNN
 F 2 "Capacitor_SMD:C_0603_1608Metric_Pad1.05x0.95mm_HandSolder" H 3300 2200 50  0001 C CNN
-F 3 "http://datasheets.avx.com/cx5r.pdf" H 3300 2200 50  0001 C CNN
+F 3 "https://static6.arrow.com/aropdfconversion/586f74e29ae0954806622435cc27099724fa32d3/grm185r60j105ke26.pdf" H 3300 2200 50  0001 C CNN
 F 4 "06033D105KAT2A" H 3300 2200 50  0001 C CNN "*Digikey"
+F 5 "GRM185R60J105KE26D" H 3300 2200 50  0001 C CNN "*Arrow"
 	1    3300 2200
 	1    0    0    -1
@@
 F 3 "http://www.jst-mfg.com/product/pdf/eng/ePH.pdf" H 4500 1850 50  0001 C CNN
 F 4 "S2B-PH-K-S(LF)(SN)" H 4750 1600 50  0000 C CNN "*Digikey"
+F 5 "S2B-PH-K-S(LF)(SN)" H 4500 1850 50  0001 C CNN "*Arrow"
 	1    4500 1850
 	1    0    0    -1
@@
 F 3 "http://ww1.microchip.com/downloads/en/DeviceDoc/20001984g.pdf" H 5950 1900 50  0001 C CNN
 F 4 "MCP73831T-2ACI/OTCT-ND" H 6100 1950 50  0001 C CNN "*Digikey"
+F 5 "MCP73831T-5ACI/OT" H 6100 1950 50  0001 C CNN "*Arrow"
 	1    6100 1950
 	1    0    0    -1
@@
 F 1 "1K" H 6800 1700 50  0000 C CNN
 F 2 "Resistor_SMD:R_0603_1608Metric_Pad1.05x0.95mm_HandSolder" H 6700 1750 50  0001 C CNN
-F 3 "https://www.bourns.com/docs/product-datasheets/CRxxxxx.pdf" H 6700 1750 50  0001 C CNN
+F 3 "https://static6.arrow.com/aropdfconversion/bc77abbb940933dbec058fcb6d36cc6b880d3e09/rn73.pdf" H 6700 1750 50  0001 C CNN
 F 4 "CR0603-FX-1001ELF" H 6700 1750 50  0001 C CNN "*Digikey"
+F 5 "RN731JTTD1001B25" H 6700 1750 50  0001 C CNN "*Arrow"
 	1    6700 1750
 	1    0    0    -1
@@
 F 1 "RED LED" V 6700 1250 50  0000 C CNN
 F 2 "LED_SMD:LED_0603_1608Metric_Pad1.05x0.95mm_HandSolder" V 6700 1500 50  0001 C CNN
-F 3 "https://www.aopled.com/AOP_PDFs/L196L-UEC.pdf" V 6700 1500 50  0001 C CNN
+F 3 "http://www.aopled.com/AOP_PDFs/L196L-UEC.pdf" V 6700 1500 50  0001 C CNN
 F 4 "L196L-UEC" H 6700 1500 50  0001 C CNN "*Digikey"
+F 5 "L196L-UEC-TR" H 6700 1500 50  0001 C CNN "*Arrow"
 	1    6700 1500
 	0    -1   -1   0
@@
 F 1 "4.7K" H 5432 2245 50  0000 R CNN
 F 2 "Resistor_SMD:R_0603_1608Metric_Pad1.05x0.95mm_HandSolder" H 5500 2200 50  0001 C CNN
-F 3 "https://www.bourns.com/docs/product-datasheets/CRxxxxx.pdf" H 5500 2200 50  0001 C CNN
+F 3 "https://static6.arrow.com/aropdfconversion/bc77abbb940933dbec058fcb6d36cc6b880d3e09/rn73.pdf" H 5500 2200 50  0001 C CNN
 F 4 "CR0603-FX-4701ELF" H 5500 2200 50  0001 C CNN "*Digikey"
+F 5 "RN731JTTD4701B25" H 5500 2200 50  0001 C CNN "*Arrow"
 	1    5500 2200
 	-1   0    0    1
@@
 P 6900 2300
 F 0 "C8" H 6992 2346 50  0000 L CNN
-F 1 "10uF 25V X7R" H 6992 2255 50  0000 L CNN
+F 1 "10uF 6.3V X5R" H 6992 2255 50  0000 L CNN
 F 2 "Capacitor_SMD:C_1210_3225Metric_Pad1.42x2.65mm_HandSolder" H 6900 2300 50  0001 C CNN
-F 3 "http://datasheets.avx.com/X7RDielectric.pdf" H 6900 2300 50  0001 C CNN
+F 3 "https://static6.arrow.com/aropdfconversion/f7a2596b5312288600ca127f041a86c0cac4c78c/grm188r60j106ke47.pdf" H 6900 2300 50  0001 C CNN
 F 4 "12103C106KAT2A" H 6900 2300 50  0001 C CNN "*Digikey"
+F 5 "GRM188R60J106KE47D" H 6900 2300 50  0001 C CNN "*Arrow"
 	1    6900 2300
 	1    0    0    -1
@@
 	3300 1150 3300 2000
 Connection ~ 3300 2000
+Text Label 1750 2000 0    50   ~ 0
+RegIn
+Text Label 2950 2000 0    50   ~ 0
+RegOut
 $EndSCHEMATC

Commit message: Changing I2C pins
Parts:
- C2, C3, C4, C8: symbol Device:C_Small -> Themu-Main-rescue:C_Small-Device
- D1: symbol Device:LED_Small_ALT -> Themu-Main-rescue:LED_Small_ALT-Device
- D2: symbol Diode:MBR340 -> Themu-Main-rescue:MBR340-Diode
- J2: symbol Connector_Generic:Conn_01x02 -> Themu-Main-rescue:Conn_01x02-Connector_Generic
- Q3: symbol Transistor_FET:DMG2301L -> Themu-Main-rescue:DMG2301L-Transistor_FET
- R6, R7, R8, R9: symbol Device:R_Small_US -> Themu-Main-rescue:R_Small_US-Device
- U2: symbol Regulator_Linear:AP2112K-3.3 -> Themu-Main-rescue:AP2112K-3.3-Regulator_Linear
- U4: symbol Battery_Management:MCP73831-2-OT -> Themu-Main-rescue:MCP73831-2-OT-Battery_Management
Changed lines of the file:
@@
 $EndDescr
 $Comp
-L Regulator_Linear:AP2112K-3.3 U2
+L Themu-Main-rescue:AP2112K-3.3-Regulator_Linear U2
 U 1 1 5F5D210A
 P 2600 2100
@@
 $EndComp
 $Comp
-L Device:R_Small_US R7
+L Themu-Main-rescue:R_Small_US-Device R7
 U 1 1 5F5D73BC
 P 2000 2100
@@
 $EndComp
 $Comp
-L Device:R_Small_US R6
+L Themu-Main-rescue:R_Small_US-Device R6
 U 1 1 5F5D82F4
 P 950 2100
@@
 $EndComp
 $Comp
-L Diode:MBR340 D2
+L Themu-Main-rescue:MBR340-Diode D2
 U 1 1 5F5DD9D5
 P 1250 2000
@@
 $EndComp
 $Comp
-L Transistor_FET:DMG2301L Q3
+L Themu-Main-rescue:DMG2301L-Transistor_FET Q3
 U 1 1 5F5E01DD
 P 1600 1500
@@
 $EndComp
 $Comp
-L Device:C_Small C2
+L Themu-Main-rescue:C_Small-Device C2
 U 1 1 5F5E1B2F
 P 1650 2350
@@
 	1700 2000 1650 2000
 $Comp
-L power:GND #PWR018
+L Themu-Main-rescue:GND-power #PWR018
 U 1 1 5F5E3B26
 P 1650 2500
@@
 $EndComp
 $Comp
-L power:VBUS #PWR016
+L Themu-Main-rescue:VBUS-power #PWR016
 U 1 1 5F5E4B32
 P 950 1150
@@
 $EndComp
 $Comp
-L power:+BATT #PWR019
+L Themu-Main-rescue:+BATT-power #PWR019
 U 1 1 5F5E597E
 P 1700 1150
@@
 $EndComp
 $Comp
-L power:GND #PWR017
+L Themu-Main-rescue:GND-power #PWR017
 U 1 1 5F5E69F8
 P 950 2500
@@
 $EndComp
 $Comp
-L power:GND #PWR020
+L Themu-Main-rescue:GND-power #PWR020
 U 1 1 5F5E74CA
 P 2600 2500
@@
 $EndComp
 $Comp
-L Device:C_Small C3
+L Themu-Main-rescue:C_Small-Device C3
 U 1 1 5F5E75DD
 P 3100 2350
@@
 $EndComp
 $Comp
-L Device:C_Small C4
+L Themu-Main-rescue:C_Small-Device C4
 U 1 1 5F5E8856
 P 3300 2200
@@
 $EndComp
 $Comp
-L power:GND #PWR021
+L Themu-Main-rescue:GND-power #PWR021
 U 1 1 5F5E8D91
 P 3100 2500
@@
 $EndComp
 $Comp
-L power:GND #PWR023
+L Themu-Main-rescue:GND-power #PWR023
 U 1 1 5F5E8FAE
 P 3300 2500
@@
 $EndComp
 $Comp
-L power:+3V3 #PWR022
+L Themu-Main-rescue:+3V3-power #PWR022
 U 1 1 5F5E9117
 P 3300 1150
@@
 	1700 1150 1700 1300
 $Comp
-L Connector_Generic:Conn_01x02 J2
+L Themu-Main-rescue:Conn_01x02-Connector_Generic J2
 U 1 1 5F5ECCBD
 P 4500 1850
@@
 $EndComp
 $Comp
-L power:+BATT #PWR024
+L Themu-Main-rescue:+BATT-power #PWR024
 U 1 1 5F5EF499
 P 4300 1500
@@
 $EndComp
 $Comp
-L power:GND #PWR025
+L Themu-Main-rescue:GND-power #PWR025
 U 1 1 5F5EFBEC
 P 4300 2350
@@
 	4300 1950 4300 2350
 $Comp
-L Battery_Management:MCP73831-2-OT U4
+L Themu-Main-rescue:MCP73831-2-OT-Battery_Management U4
 U 1 1 5F5F1703
 P 6100 1950
@@
 $EndComp
 $Comp
-L Device:R_Small_US R9
+L Themu-Main-rescue:R_Small_US-Device R9
 U 1 1 5F5F379D
 P 6700 1750
@@
 $EndComp
 $Comp
-L Device:LED_Small_ALT D1
+L Themu-Main-rescue:LED_Small_ALT-Device D1
 U 1 1 5F5F5CC9
 P 6700 1500
@@
 $EndComp
 $Comp
-L power:VBUS #PWR027
+L Themu-Main-rescue:VBUS-power #PWR027
 U 1 1 5F5FC6D9
 P 6700 1300
@@
 	6700 2050 6500 2050
 $Comp
-L Device:R_Small_US R8
+L Themu-Main-rescue:R_Small_US-Device R8
 U 1 1 5F5FD9AD
 P 5500 2200
@@
 $EndComp
 $Comp
-L power:GND #PWR026
+L Themu-Main-rescue:GND-power #PWR026
 U 1 1 5F5FF071
 P 6100 2400
@@
 $EndComp
 $Comp
-L Device:C_Small C8
+L Themu-Main-rescue:C_Small-Device C8
 U 1 1 5F5FFAAE
 P 6900 2300
@@
 $EndComp
 $Comp
-L power:GND #PWR029
+L Themu-Main-rescue:GND-power #PWR029
 U 1 1 5F6012DA
 P 6900 2400
@@
 5K = 200mA\n2K = 500mA\n1K = 1000mA\n
 $Comp
-L power:+BATT #PWR028
+L Themu-Main-rescue:+BATT-power #PWR028
 U 1 1 5F6A9BEF
 P 6900 2100
@@
 Connection ~ 6900 2200
 $Comp
-L power:PWR_FLAG #FLG0101
+L Themu-Main-rescue:PWR_FLAG-power #FLG0101
 U 1 1 5F73E5D7
 P 2100 2000
