File: Main_Board/Power.sch (KiCad schematic (older format))
At the start: 14 parts, among them J2 Conn_01x02, Q3 DMG2305U, U2 AP2112K-3.3, U4 MCP73831-2-OT

Commit message: Changing I2C pins (continue)
Parts:
- C2, C3, C4, C8: symbol Themu-Main-rescue:C_Small-Device -> Device:C_Small
- D1: symbol Themu-Main-rescue:LED_Small_ALT-Device -> Device:LED_Small_ALT
- D2: symbol Themu-Main-rescue:MBR340-Diode -> Diode:MBR340
- J2: symbol Themu-Main-rescue:Conn_01x02-Connector_Generic -> Connector_Generic:Conn_01x02
- Q3: symbol Themu-Main-rescue:DMG2301L-Transistor_FET -> Transistor_FET:DMG2301L
- R6, R7, R8, R9: symbol Themu-Main-rescue:R_Small_US-Device -> Device:R_Small_US
- U2: symbol Themu-Main-rescue:AP2112K-3.3-Regulator_Linear -> Regulator_Linear:AP2112K-3.3
- U4: symbol Themu-Main-rescue:MCP73831-2-OT-Battery_Management -> Battery_Management:MCP73831-2-OT
Changed lines of the file:
@@
 $EndDescr
 $Comp
-L Themu-Main-rescue:AP2112K-3.3-Regulator_Linear U2
+L Regulator_Linear:AP2112K-3.3 U2
 U 1 1 5F5D210A
 P 2600 2100
@@
 $EndComp
 $Comp
-L Themu-Main-rescue:R_Small_US-Device R7
+L Device:R_Small_US R7
 U 1 1 5F5D73BC
 P 2000 2100
@@
 $EndComp
 $Comp
-L Themu-Main-rescue:R_Small_US-Device R6
+L Device:R_Small_US R6
 U 1 1 5F5D82F4
 P 950 2100
@@
 $EndComp
 $Comp
-L Themu-Main-rescue:MBR340-Diode D2
+L Diode:MBR340 D2
 U 1 1 5F5DD9D5
 P 1250 2000
@@
 $EndComp
 $Comp
-L Themu-Main-rescue:DMG2301L-Transistor_FET Q3
+L Transistor_FET:DMG2301L Q3
 U 1 1 5F5E01DD
 P 1600 1500
@@
 $EndComp
 $Comp
-L Themu-Main-rescue:C_Small-Device C2
+L Device:C_Small C2
 U 1 1 5F5E1B2F
 P 1650 2350
@@
 	1700 2000 1650 2000
 $Comp
-L Themu-Main-rescue:GND-power #PWR018
+L power:GND #PWR018
 U 1 1 5F5E3B26
 P 1650 2500
@@
 $EndComp
 $Comp
-L Themu-Main-rescue:VBUS-power #PWR016
+L power:VBUS #PWR016
 U 1 1 5F5E4B32
 P 950 1150
@@
 $EndComp
 $Comp
-L Themu-Main-rescue:+BATT-power #PWR019
+L power:+BATT #PWR019
 U 1 1 5F5E597E
 P 1700 1150
@@
 $EndComp
 $Comp
-L Themu-Main-rescue:GND-power #PWR017
+L power:GND #PWR017
 U 1 1 5F5E69F8
 P 950 2500
@@
 $EndComp
 $Comp
-L Themu-Main-rescue:GND-power #PWR020
+L power:GND #PWR020
 U 1 1 5F5E74CA
 P 2600 2500
@@
 $EndComp
 $Comp
-L Themu-Main-rescue:C_Small-Device C3
+L Device:C_Small C3
 U 1 1 5F5E75DD
 P 3100 2350
@@
 $EndComp
 $Comp
-L Themu-Main-rescue:C_Small-Device C4
+L Device:C_Small C4
 U 1 1 5F5E8856
 P 3300 2200
@@
 $EndComp
 $Comp
-L Themu-Main-rescue:GND-power #PWR021
+L power:GND #PWR021
 U 1 1 5F5E8D91
 P 3100 2500
@@
 $EndComp
 $Comp
-L Themu-Main-rescue:GND-power #PWR023
+L power:GND #PWR023
 U 1 1 5F5E8FAE
 P 3300 2500
@@
 $EndComp
 $Comp
-L Themu-Main-rescue:+3V3-power #PWR022
+L power:+3V3 #PWR022
 U 1 1 5F5E9117
 P 3300 1150
@@
 	1700 1150 1700 1300
 $Comp
-L Themu-Main-rescue:Conn_01x02-Connector_Generic J2
+L Connector_Generic:Conn_01x02 J2
 U 1 1 5F5ECCBD
 P 4500 1850
@@
 $EndComp
 $Comp
-L Themu-Main-rescue:+BATT-power #PWR024
+L power:+BATT #PWR024
 U 1 1 5F5EF499
 P 4300 1500
@@
 $EndComp
 $Comp
-L Themu-Main-rescue:GND-power #PWR025
+L power:GND #PWR025
 U 1 1 5F5EFBEC
 P 4300 2350
@@
 	4300 1950 4300 2350
 $Comp
-L Themu-Main-rescue:MCP73831-2-OT-Battery_Management U4
+L Battery_Management:MCP73831-2-OT U4
 U 1 1 5F5F1703
 P 6100 1950
@@
 $EndComp
 $Comp
-L Themu-Main-rescue:R_Small_US-Device R9
+L Device:R_Small_US R9
 U 1 1 5F5F379D
 P 6700 1750
@@
 $EndComp
 $Comp
-L Themu-Main-rescue:LED_Small_ALT-Device D1
+L Device:LED_Small_ALT D1
 U 1 1 5F5F5CC9
 P 6700 1500
@@
 $EndComp
 $Comp
-L Themu-Main-rescue:VBUS-power #PWR027
+L power:VBUS #PWR027
 U 1 1 5F5FC6D9
 P 6700 1300
@@
 	6700 2050 6500 2050
 $Comp
-L Themu-Main-rescue:R_Small_US-Device R8
+L Device:R_Small_US R8
 U 1 1 5F5FD9AD
 P 5500 2200
@@
 $EndComp
 $Comp
-L Themu-Main-rescue:GND-power #PWR026
+L power:GND #PWR026
 U 1 1 5F5FF071
 P 6100 2400
@@
 $EndComp
 $Comp
-L Themu-Main-rescue:C_Small-Device C8
+L Device:C_Small C8
 U 1 1 5F5FFAAE
 P 6900 2300
@@
 $EndComp
 $Comp
-L Themu-Main-rescue:GND-power #PWR029
+L power:GND #PWR029
 U 1 1 5F6012DA
 P 6900 2400
@@
 5K = 200mA\n2K = 500mA\n1K = 1000mA\n
 $Comp
-L Themu-Main-rescue:+BATT-power #PWR028
+L power:+BATT #PWR028
 U 1 1 5F6A9BEF
 P 6900 2100
@@
 Connection ~ 6900 2200
 $Comp
-L Themu-Main-rescue:PWR_FLAG-power #FLG0101
+L power:PWR_FLAG #FLG0101
 U 1 1 5F73E5D7
 P 2100 2000

Commit message: C2, C3, C8 and C14 footprints and packages changed from 1210 to 0603 (#11)
Parts:
- C2, C3, C8: footprint Capacitor_SMD:C_1210_3225Metric_Pad1.42x2.65mm_HandSolder -> Capacitor_SMD:C_0603_1608Metric_Pad1.08x0.95mm_HandSolder
Changed lines of the file:
@@
 F 0 "C2" H 1742 2396 50  0000 L CNN
 F 1 "10uF 6.3V X5R" H 1742 2305 50  0000 L CNN
-F 2 "Capacitor_SMD:C_1210_3225Metric_Pad1.42x2.65mm_HandSolder" H 1650 2350 50  0001 C CNN
+F 2 "Capacitor_SMD:C_0603_1608Metric_Pad1.08x0.95mm_HandSolder" H 1650 2350 50  0001 C CNN
 F 3 "https://static6.arrow.com/aropdfconversion/f7a2596b5312288600ca127f041a86c0cac4c78c/grm188r60j106ke47.pdf" H 1650 2350 50  0001 C CNN
 F 4 "12103C106KAT2A" H 1650 2350 50  0001 C CNN "*Digikey"
@@
 F 0 "C3" H 3400 2350 50  0000 L CNN
 F 1 "10uF 6.3V X5R" H 3550 2350 50  0000 L CNN
-F 2 "Capacitor_SMD:C_1210_3225Metric_Pad1.42x2.65mm_HandSolder" H 3100 2350 50  0001 C CNN
+F 2 "Capacitor_SMD:C_0603_1608Metric_Pad1.08x0.95mm_HandSolder" H 3100 2350 50  0001 C CNN
 F 3 "https://static6.arrow.com/aropdfconversion/f7a2596b5312288600ca127f041a86c0cac4c78c/grm188r60j106ke47.pdf" H 3100 2350 50  0001 C CNN
 F 4 "12103C106KAT2A" H 3100 2350 50  0001 C CNN "*Digikey"
@@
 F 0 "C8" H 6992 2346 50  0000 L CNN
 F 1 "10uF 6.3V X5R" H 6992 2255 50  0000 L CNN
-F 2 "Capacitor_SMD:C_1210_3225Metric_Pad1.42x2.65mm_HandSolder" H 6900 2300 50  0001 C CNN
+F 2 "Capacitor_SMD:C_0603_1608Metric_Pad1.08x0.95mm_HandSolder" H 6900 2300 50  0001 C CNN
 F 3 "https://static6.arrow.com/aropdfconversion/f7a2596b5312288600ca127f041a86c0cac4c78c/grm188r60j106ke47.pdf" H 6900 2300 50  0001 C CNN
 F 4 "12103C106KAT2A" H 6900 2300 50  0001 C CNN "*Digikey"
